File: Stepper.kicad_sch (KiCad schematic)
At the start: 56 parts, among them J3 DE9_Socket_MountingHoles, J6 DE9_Socket_MountingHoles, Q1 2N7002KQ-7, Q13 2N7002KQ-7, Q2 2N7002KQ-7, Q3 2N7002KQ-7, Q4 2N7002KQ-7, Q5 2N7002KQ-7, U10 ISO6762DWR, U11 TPD2E2U06QDBZRQ1, U12 TPD2E2U06QDBZRQ1, U18 ISO6762DWR, U19 TPD2E2U06QDBZRQ1, U20 TPD2E2U06QDBZRQ1

Commit message: Redesign schematic for dual motor encoders
Connections:
- net LH_ENC_POS_PRESET renamed PORT_ENC_POS_PRESET
- net LH_ENC_PRESET renamed PORT_ENC_PRESET
- net LH_STR8_5V_FIELD renamed PORT_STR8_5V_FIELD
- net LH_STR8_DIR_CMD renamed PORT_STR8_DIR_CMD
- net LH_STR8_DISABLE renamed PORT_STR8_DISABLE
- net LH_STR8_FAULT renamed PORT_STR8_FAULT
- net LH_STR8_FAULT_RAW renamed PORT_STR8_FAULT_RAW
- net LH_STR8_STEP_CMD renamed PORT_STR8_STEP_CMD
- net RH_ENC_POS_PRESET renamed STAR_ENC_POS_PRESET
- net RH_ENC_PRESET renamed STAR_ENC_PRESET
- net RH_STR8_5V_FIELD renamed STAR_STR8_5V_FIELD
- net RH_STR8_DIR_CMD renamed STAR_STR8_DIR_CMD
- net RH_STR8_DISABLE renamed STAR_STR8_DISABLE
- net RH_STR8_FAULT renamed STAR_STR8_FAULT
- net RH_STR8_FAULT_RAW renamed STAR_STR8_FAULT_RAW
- net RH_STR8_STEP_CMD renamed STAR_STR8_STEP_CMD
Other:
- note added: "Digital isolator"
- note added: "Signal ESD protection"
Changed lines of the file:
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@@
 	(title_block
 		(title "Elevation Control_Gigabit")
-		(date "2026-09-01")
-		(rev "Sep_2026_V1")
+		(date "2026-10-03")
+		(rev "P3 REVIEW")
 		(company "Starspec")
 		(comment 4 "Mauro M. Coutinho")
 	)
+	(text "Signal ESD protection"
+		(exclude_from_sim no)
+		(at 257.81 175.26 0)
+		(effects
+			(font
+				(size 1.27 1.27)
+			)
+		)
+	)
 	(text "STR8 CONTROL - STM32 SIGNALS ACTIVE HIGH\nPE9/TIM1_CH1 STEP: idle LOW; generate HIGH pulses, minimum 3 us.\nPE11 DIR: set direction before starting STEP pulses.\nPE13 STR8_DISABLE: HIGH = motor disabled; keep HIGH during reset/startup.\nPE14 STR8_FAULT: HIGH = fault; stop STEP and assert STR8_DISABLE.\nStartup: DISABLE HIGH -> configure STEP/DIR -> DISABLE LOW. STR8 S4 filter: 150 kHz.\n"
 		(exclude_from_sim no)
@@
 		)
 	)
+	(text "Signal ESD protection"
+		(exclude_from_sim no)
+		(at 257.81 68.58 0)
+		(effects
+			(font
+				(size 1.27 1.27)
+			)
+		)
+	)
+	(text "Digital isolator"
+		(exclude_from_sim no)
+		(at 95.25 176.53 0)
+		(effects
+			(font
+				(size 1.27 1.27)
+			)
+		)
+	)
+	(text "Digital isolator"
+		(exclude_from_sim no)
+		(at 95.25 69.85 0)
+		(effects
+			(font
+				(size 1.27 1.27)
+			)
+		)
+	)
 	(junction
 		(at 218.44 68.58)
@@
 	(wire
 		(pts
-			(xy 30.48 104.14) (xy 59.69 104.14)
+			(xy 33.02 104.14) (xy 59.69 104.14)
 		)
 		(stroke
@@
 		)
 	)
-	(global_label "RH_ENC_POS_PRESET"
+	(global_label "STAR_ENC_POS_PRESET"
 		(shape input)
 		(at 116.84 200.66 0)
@@
 		)
 	)
-	(global_label "LH_STR8_5V_FIELD"
+	(global_label "PORT_STR8_5V_FIELD"
 		(shape input)
 		(at 207.01 58.42 180)
@@
 		)
 	)
-	(global_label "LH_STR8_FAULT_RAW"
+	(global_label "PORT_STR8_FAULT_RAW"
 		(shape input)
 		(at 125.73 96.52 270)
@@
 		)
 	)
-	(global_label "RH_STR8_5V_FIELD"
+	(global_label "STAR_STR8_5V_FIELD"
 		(shape input)
 		(at 213.36 207.01 270)
@@
 		)
 	)
-	(global_label "RH_STR8_5V_FIELD"
+	(global_label "STAR_STR8_5V_FIELD"
 		(shape input)
 		(at 213.36 200.66 180)
@@
 		)
 	)
-	(global_label "LH_STR8_5V_FIELD"
+	(global_label "PORT_STR8_5V_FIELD"
 		(shape input)
 		(at 213.36 100.33 270)
@@
 		)
 	)
-	(global_label "RH_STR8_5V_FIELD"
+	(global_label "STAR_STR8_5V_FIELD"
 		(shape input)
 		(at 213.36 190.5 180)
@@
 		)
 	)
-	(global_label "LH_STR8_FAULT_RAW"
+	(global_label "PORT_STR8_FAULT_RAW"
 		(shape input)
 		(at 189.23 96.52 270)
@@
 		)
 	)
-	(global_label "RH_STR8_FAULT_RAW"
+	(global_label "STAR_STR8_FAULT_RAW"
 		(shape input)
 		(at 125.73 203.2 270)
@@
 		)
 	)
-	(global_label "LH_STR8_5V_FIELD"
+	(global_label "PORT_STR8_5V_FIELD"
 		(shape input)
 		(at 213.36 83.82 180)
@@
 		)
 	)
-	(global_label "RH_STR8_5V_FIELD"
+	(global_label "STAR_STR8_5V_FIELD"
 		(shape input)
 		(at 207.01 165.1 180)
@@
 		)
 	)
-	(global_label "LH_STR8_5V_FIELD"
+	(global_label "PORT_STR8_5V_FIELD"
 		(shape input)
 		(at 213.36 88.9 180)
@@
 		)
 	)
-	(global_label "LH_ENC_POS_PRESET"
+	(global_label "PORT_ENC_POS_PRESET"
 		(shape input)
 		(at 116.84 93.98 0)
@@
 		)
 	)
-	(global_label "LH_STR8_5V_FIELD"
+	(global_label "PORT_STR8_5V_FIELD"
 		(shape input)
 		(at 213.36 93.98 180)
@@
 		)
 	)
-	(global_label "RH_STR8_5V_FIELD"
+	(global_label "STAR_STR8_5V_FIELD"
 		(shape input)
 		(at 213.36 195.58 180)
@@
 		)
 	)
-	(global_label "RH_STR8_FAULT_RAW"
+	(global_label "STAR_STR8_FAULT_RAW"
 		(shape input)
 		(at 189.23 203.2 270)
@@
 		)
 	)
-	(hierarchical_label "LH_STR8_DIR_CMD"
+	(hierarchical_label "PORT_STR8_DIR_CMD"
 		(shape input)
 		(at 48.26 81.28 180)
@@
 		)
 	)
-	(hierarchical_label "RH_STR8_DIR_CMD"
+	(hierarchical_label "STAR_STR8_DIR_CMD"
 		(shape input)
 		(at 48.26 187.96 180)
@@
 		)
 	)
-	(hierarchical_label "LH_STR8_FAULT"
+	(hierarchical_label "PORT_STR8_FAULT"
 		(shape output)
 		(at 60.96 120.65 180)
@@
 		)
 	)
-	(hierarchical_label "RH_STR8_STEP_CMD"
+	(hierarchical_label "STAR_STR8_STEP_CMD"
 		(shape input)
 		(at 49.53 177.8 180)
@@
 		)
 	)
-	(hierarchical_label "LH_ENC_PRESET"
+	(hierarchical_label "PORT_ENC_PRESET"
 		(shape input)
-		(at 30.48 104.14 180)
+		(at 33.02 104.14 180)
 		(effects
 			(font
@@
 		)
 	)
-	(hierarchical_label "RH_ENC_PRESET"
+	(hierarchical_label "STAR_ENC_PRESET"
 		(shape input)
 		(at 35.56 212.09 180)
@@
 		)
 	)
-	(hierarchical_label "RH_STR8_FAULT"
+	(hierarchical_label "STAR_STR8_FAULT"
 		(shape output)
 		(at 60.96 224.79 180)
@@
 		)
 	)
-	(hierarchical_label "LH_STR8_DISABLE"
+	(hierarchical_label "PORT_STR8_DISABLE"
 		(shape input)
 		(at 46.99 91.44 180)
@@
 		)
 	)
-	(hierarchical_label "RH_STR8_DISABLE"
+	(hierarchical_label "STAR_STR8_DISABLE"
 		(shape input)
 		(at 46.99 198.12 180)
@@
 		)
 	)
-	(hierarchical_label "LH_STR8_STEP_CMD"
+	(hierarchical_label "PORT_STR8_STEP_CMD"
 		(shape input)
 		(at 49.53 71.12 180)
@@
 		(property "ALT_LCSC" "C5216384"
 			(at 74.93 83.82 0)
-			(effects (font (size 1.27 1.27)) (hide yes))
+			(effects
+				(font
+					(size 1.27 1.27)
+				)
+				(hide yes)
+			)
 		)
 		(property "ALT_MANUFACTURER_PART_NUMBER" "ISO6762QDWRQ1"
 			(at 74.93 83.82 0)
-			(effects (font (size 1.27 1.27)) (hide yes))
+			(effects
+				(font
+					(size 1.27 1.27)
+				)
+				(hide yes)
+			)
 		)
 		(pin "8"
@@
 		(property "ALT_LCSC" "C5216384"
 			(at 74.93 190.5 0)
-			(effects (font (size 1.27 1.27)) (hide yes))
+			(effects
+				(font
+					(size 1.27 1.27)
+				)
+				(hide yes)
+			)
 		)
 		(property "ALT_MANUFACTURER_PART_NUMBER" "ISO6762QDWRQ1"
 			(at 74.93 190.5 0)
-			(effects (font (size 1.27 1.27)) (hide yes))
+			(effects
+				(font
+					(size 1.27 1.27)
+				)
+				(hide yes)
+			)
 		)
 		(pin "8"

Commit message: Preserve P5 equal-size placement, controller stack and native BOM
Parts:
- C37, C42, C69, C72: Assembly (none) -> FIT; BOM Status (none) -> PART IDENTIFIED; sourcing/footprint review pending; Footprint Status (none) -> Assigned; drawing/pad verification pending; Function (none) -> Unpolarized capacitor; JLCPCB Status (none) -> Historical ID; recheck exact part and assembly availability; MPN (none) -> CL31B105KCHNNNE; Supplier Data Checked (none) -> UNDATED legacy record; Supplier Source (none) -> Legacy schematic record; exact supplier listing verificatio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; Temp Basis (none) -> Legacy rating; ambient/junction basis unverified; Temp Max (degC) (none) -> 125; Temp Min (degC) (none) -> -55; Temp Source (none) -> Legacy schematic field; primary-source verification pending; Temp Status (none) -> Inherited rating; system requirement pending
- C38, C40, C53, C70, C71, C97: Assembly (none) -> FIT; BOM Status (none) -> PART IDENTIFIED; sourcing/footprint review pending; Footprint Status (none) -> Assigned; drawing/pad verification pending; Function (none) -> Unpolarized capacitor; JLCPCB Status (none) -> Historical ID; recheck exact part and assembly availability; MPN (none) -> CL21B104KCFNNNE; Supplier Data Checked (none) -> UNDATED legacy record; Supplier Source (none) -> Legacy schematic record; exact supplier listing verificatio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; Temp Basis (none) -> Legacy rating; ambient/junction basis unverified; Temp Max (degC) (none) -> 125; Temp Min (degC) (none) -> -55; Temp Source (none) -> Legacy schematic field; primary-source verification pending; Temp Status (none) -> Inherited rating; system requirement pending
- C51, C96: Assembly (none) -> FIT; BOM Status (none) -> PART IDENTIFIED; sourcing/footprint review pending; Footprint Status (none) -> Assigned; drawing/pad verification pending; Function (none) -> Unpolarized capacitor; JLCPCB Status (none) -> Historical ID; recheck exact part and assembly availability; MPN (none) -> CL21B103KCANNNC; Supplier Data Checked (none) -> UNDATED legacy record; Supplier Source (none) -> Legacy schematic record; exact supplier listing verificatio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; Temp Basis (none) -> Legacy rating; ambient/junction basis unverified; Temp Max (degC) (none) -> 125; Temp Min (degC) (none) -> -55; Temp Source (none) -> Legacy schematic field; primary-source verification pending; Temp Status (none) -> Inherited rating; system requirement pending
- C52, C98: Assembly (none) -> FIT; BOM Status (none) -> PART IDENTIFIED; sourcing/footprint review pending; Footprint Status (none) -> Assigned; drawing/pad verification pending; Function (none) -> Unpolarized capacitor; JLCPCB Status (none) -> Historical ID; recheck exact part and assembly availability; MPN (none) -> CL32B475KCVZNWE; Supplier Data Checked (none) -> UNDATED legacy record; Supplier Source (none) -> Legacy schematic record; exact supplier listing verificatio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; Temp Basis (none) -> Legacy rating; ambient/junction basis unverified; Temp Max (degC) (none) -> 125; Temp Min (degC) (none) -> -55; Temp Source (none) -> Legacy schematic field; primary-source verification pending; Temp Status (none) -> Inherited rating; system requirement pending
- D1, D4: Assembly (none) -> FIT; BOM Status (none) -> PART IDENTIFIED; sourcing/footprint review pending; Footprint Status (none) -> Assigned; drawing/pad verification pending; Function (none) -> TPD1E10B06DPYR; JLCPCB Status (none) -> Historical ID; recheck exact part and assembly availability; MPN (none) -> TPD1E10B06DPYR; Supplier Data Checked (none) -> UNDATED legacy record; Supplier Source (none) -> Legacy schematic record; exact supplier listing verificatio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; Temp Basis (none) -> Legacy rating; ambient/junction basis unverified; Temp Max (degC) (none) -> 125; Temp Min (degC) (none) -> -40; Temp Source (none) -> Legacy schematic field; primary-source verification pending; Temp Status (none) -> Inherited rating; system requirement pending
- J3, J6: Assembly (none) -> FIT; BOM Review (none) -> Same MPN as existing DE9 connectors. Verify exact pin grid,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; BOM Status (none) -> PART IDENTIFIED; sourcing/footprint review pending; Footprint Status (none) -> REVIEW: compare exact TE drawing to generic KiCad footprint; Function (none) -> DE9 female right-angle PCB connector; JLCPCB Library (none) -> UNVERIFIED; JLCPCB Status (none) -> LCSC exact match; JLC assembly availability unverified; MPN (none) -> 5747844-4; Supplier Data Checked (none) -> 2026-10-03; Supplier Source (none) -> https://www.lcsc.com/de/product-detail/C305941.html; Temp Basis (none) -> Operating; Temp Checked (none) -> 2026-10-03; Temp Max (degC) (none) -> 105; Temp Min (degC) (none) -> -55; Temp Source (none) -> https://www.te.com/en/product-5747844-4.html; Temp Status (none) -> Manufacturer rating recorded; system requirement pending
- Q1, Q13, Q2, Q3, Q4, Q5: Assembly (none) -> FIT; BOM Review (none) -> Legacy datasheet points to onsemi NDS7002A rather than sele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; BOM Status (none) -> REVIEW: legacy datasheet/manufacturer mismatch; Footprint Status (none) -> Assigned; drawing/pad verification pending; Function (none) -> 0.115A Id, 60V Vds, N-Channel MOSFET, SOT-23; JLCPCB Status (none) -> Historical ID; recheck exact part and assembly availability; MPN (none) -> 2N7002KQ-7; Supplier Data Checked (none) -> UNDATED legacy record; Supplier Source (none) -> Legacy schematic record; exact supplier listing verificatio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; Temp Basis (none) -> Legacy rating; ambient/junction basis unverified; Temp Max (degC) (none) -> 150; Temp Min (degC) (none) -> -55; Temp Source (none) -> Legacy schematic field; primary-source verification pending; Temp Status (none) -> Legacy rating unverified; exact manufacturer datasheet requ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
- R27, R55: Assembly (none) -> FIT; BOM Status (none) -> PART IDENTIFIED; sourcing/footprint review pending; Footprint Status (none) -> Assigned; drawing/pad verification pending; Function (none) -> Resistor; JLCPCB Status (none) -> Historical ID; recheck exact part and assembly availability; MPN (none) -> RC0805FR-074K7L; Supplier Data Checked (none) -> UNDATED legacy record; Supplier Source (none) -> Legacy schematic record; exact supplier listing verificatio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; Temp Basis (none) -> Legacy rating; ambient/junction basis unverified; Temp Max (degC) (none) -> 155; Temp Min (degC) (none) -> -55; Temp Source (none) -> Legacy schematic field; primary-source verification pending; Temp Status (none) -> Inherited rating; system requirement pending
- R28, R29, R36, R37, R45, R46, R47, R48, R57, R58: Assembly (none) -> FIT; BOM Status (none) -> PART IDENTIFIED; sourcing/footprint review pending; Footprint Status (none) -> Assigned; drawing/pad verification pending; Function (none) -> Resistor; JLCPCB Status (none) -> Historical ID; recheck exact part and assembly availability; MPN (none) -> RC0805FR-0710KL; Supplier Data Checked (none) -> UNDATED legacy record; Supplier Source (none) -> Legacy schematic record; exact supplier listing verificatio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; Temp Basis (none) -> Legacy rating; ambient/junction basis unverified; Temp Max (degC) (none) -> 155; Temp Min (degC) (none) -> -55; Temp Source (none) -> Legacy schematic field; primary-source verification pending; Temp Status (none) -> Inherited rating; system requirement pending
- R30, R31, R32, R49, R50, R51: Assembly (none) -> FIT; BOM Status (none) -> PART IDENTIFIED; sourcing/footprint review pending; Footprint Status (none) -> Assigned; drawing/pad verification pending; Function (none) -> Resistor; JLCPCB Status (none) -> Historical ID; recheck exact part and assembly availability; MPN (none) -> RC0805FR-07100RL; Supplier Data Checked (none) -> UNDATED legacy record; Supplier Source (none) -> Legacy schematic record; exact supplier listing verificatio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; Temp Basis (none) -> Legacy rating; ambient/junction basis unverified; Temp Max (degC) (none) -> 155; Temp Min (degC) (none) -> -55; Temp Source (none) -> Legacy schematic field; primary-source verification pending; Temp Status (none) -> Inherited rating; system requirement pending
- R33, R34, R35, R52, R53, R54: Assembly (none) -> FIT; BOM Status (none) -> PART IDENTIFIED; sourcing/footprint review pending; Footprint Status (none) -> Assigned; drawing/pad verification pending; Function (none) -> Resistor; JLCPCB Status (none) -> Historical ID; recheck exact part and assembly availability; MPN (none) -> RC0805FR-0747KL; Supplier Data Checked (none) -> UNDATED legacy record; Supplier Source (none) -> Legacy schematic record; exact supplier listing verificatio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; Temp Basis (none) -> Legacy rating; ambient/junction basis unverified; Temp Max (degC) (none) -> 155; Temp Min (degC) (none) -> -55; Temp Source (none) -> Legacy schematic field; primary-source verification pending; Temp Status (none) -> Inherited rating; system requirement pending
- R38, R56: Assembly (none) -> FIT; BOM Status (none) -> PART IDENTIFIED; sourcing/footprint review pending; Footprint Status (none) -> Assigned; drawing/pad verification pending; Function (none) -> Resistor; JLCPCB Status (none) -> Historical ID; recheck exact part and assembly availability; MPN (none) -> 352210RFT; Supplier Data Checked (none) -> UNDATED legacy record; Supplier Source (none) -> Legacy schematic record; exact supplier listing verificatio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; Temp Basis (none) -> Legacy rating; ambient/junction basis unverified; Temp Max (degC) (none) -> 155; Temp Min (degC) (none) -> -55; Temp Source (none) -> Legacy schematic field; primary-source verification pending; Temp Status (none) -> Inherited rating; system requirement pending
- U10, U18: Assembly (none) -> FIT; BOM Status (none) -> PART IDENTIFIED; sourcing/footprint review pending; Footprint Status (none) -> Assigned; drawing/pad verification pending; Function (none) -> ISO6762DWR; JLCPCB Status (none) -> Historical ID; recheck exact part and assembly availability; MPN (none) -> ISO6762DWR; Supplier Data Checked (none) -> UNDATED legacy record; Supplier Source (none) -> Legacy schematic record; exact supplier listing verificatio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; Temp Basis (none) -> Legacy rating; ambient/junction basis unverified; Temp Max (degC) (none) -> 125; Temp Min (degC) (none) -> -40; Temp Source (none) -> Legacy schematic field; primary-source verification pending; Temp Status (none) -> Inherited rating; system requirement pending
- U11, U12, U19, U20: Assembly (none) -> FIT; BOM Status (none) -> PART IDENTIFIED; sourcing/footprint review pending; Footprint Status (none) -> Assigned; drawing/pad verification pending; Function (none) -> Automotive Dual-Channel High-Speed ESD Protection Device; JLCPCB Status (none) -> Historical ID; recheck exact part and assembly availability; MPN (none) -> TPD2E2U06QDBZRQ1; Supplier Data Checked (none) -> UNDATED legacy record; Supplier Source (none) -> Legacy schematic record; exact supplier listing verificatio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; Temp Basis (none) -> Legacy rating; ambient/junction basis unverified; Temp Max (degC) (none) -> 125; Temp Min (degC) (none) -> -40; Temp Source (none) -> Legacy schematic field; primary-source verification pending; Temp Status (none) -> Inherited rating; system requirement pending
