File: ADS1115.kicad_sch (KiCad schematic)
At the start: 11 parts, among them U21 ADS1115BQDGSRQ1, U24 ISO1540DR

Commit message: Redesign schematic for dual motor encoders
Parts:
- added C190, C191: 100n, Capacitor_SMD:C_0805_2012Metric, symbol Pivot_Reviewed:C
- added R180, R181: 10k 0.1%, Resistor_SMD:R_0805_2012Metric, symbol Pivot_Reviewed:R
- added R182, R183: 1k, Resistor_SMD:R_0805_2012Metric, symbol Pivot_Reviewed:R
- added TH1, TH2: 10k NTC / 1206, Resistor_SMD:R_1206_3216Metric, symbol Pivot_Reviewed:Thermistor_NTC
Connections:
- net +5V_BRAKE: now also TH1.1, TH2.1
- net GND_BRAKE: now also C190.2, C191.2, R180.2, R181.2
- net TEMP_BOARD: now reaches U21.6 (AIN2)
- net TEMP_BOARD: now also C190.1, R182.2
- net TEMP_POWER: now reaches U21.7 (AIN3)
- net TEMP_POWER: now also C191.1, R183.2
- net LH_BRAKE_CURR renamed PORT_BRAKE_CURR
- net RH_BRAKE_CURR renamed STAR_BRAKE_CURR
- new net: R180.1, R182.1, TH1.2
- new net: R181.1, R183.1, TH2.2
- no-connect marks 3 -> 1
Other:
- note added: "16-bit, 4-channel ADC"
- note added: "Board temperature"
- note added: "I2C digital isolator"
- note added: "ONBOARD TEMPERATURE"
- note added: "Power-area temperature"
- note added: "TH1 / TH2: two-pad 1206 thermistors, mounted on this PCB. Place TH1 away from heat sources; TH2 near the selected power hot spot. Both circuits stay in the +5V_BRAKE / GND_BRAKE domain; preserve isolation clearances."
- note added: "U21 AIN2 = TEMP_BOARD; AIN3 = TEMP_POWER. No added ICs or I2C addresses. Firmware: use +/-6.144 V range for AIN2/3; keep brake AIN0/1 at +/-4.096 V. Use TDK R/T curve 1010 and calibrated excitation voltage; voltage rises with temperature. Readings require the brake supply. Placement, calibration and cold testing remain to be done."

Commit message: Preserve P5 equal-size placement, controller stack and native BOM
Parts:
- C190, C191: Assembly (none) -> FIT; BOM Status (none) -> PART IDENTIFIED; sourcing/footprint review pending; Footprint Status (none) -> Assigned; drawing/pad verification pending; Function (none) -> Unpolarized capacitor; JLCPCB Status (none) -> Historical ID; recheck exact part and assembly availability; LCSC (none) -> C28233; MPN (none) -> CL21B104KCFNNNE; Manufacturer (none) -> Samsung Electro-Mechanics; Operating Temperature (none) -> -55 to +125 C; Supplier Data Checked (none) -> UNDATED legacy record; Supplier Source (none) -> Legacy schematic record; exact supplier listing verificatio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; Temp Basis (none) -> Legacy rating; ambient/junction basis unverified; Temp Max (degC) (none) -> 125; Temp Min (degC) (none) -> -55; Temp Source (none) -> Legacy schematic field; primary-source verification pending; Temp Status (none) -> Inherited rating; system requirement pending
- C87, C89: Assembly (none) -> FIT; BOM Status (none) -> PART IDENTIFIED; sourcing/footprint review pending; Footprint Status (none) -> Assigned; drawing/pad verification pending; Function (none) -> Unpolarized capacitor; JLCPCB Status (none) -> Historical ID; recheck exact part and assembly availability; MPN (none) -> CL32B106KBJNFNE; Supplier Data Checked (none) -> UNDATED legacy record; Supplier Source (none) -> Legacy schematic record; exact supplier listing verificatio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; Temp Basis (none) -> Legacy rating; ambient/junction basis unverified; Temp Max (degC) (none) -> 125; Temp Min (degC) (none) -> -55; Temp Source (none) -> Legacy schematic field; primary-source verification pending; Temp Status (none) -> Inherited rating; system requirement pending
- C88, C90, C91: Assembly (none) -> FIT; BOM Status (none) -> PART IDENTIFIED; sourcing/footprint review pending; Footprint Status (none) -> Assigned; drawing/pad verification pending; Function (none) -> Unpolarized capacitor; JLCPCB Status (none) -> Historical ID; recheck exact part and assembly availability; MPN (none) -> CL21B104KCFNNNE; Supplier Data Checked (none) -> UNDATED legacy record; Supplier Source (none) -> Legacy schematic record; exact supplier listing verificatio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; Temp Basis (none) -> Legacy rating; ambient/junction basis unverified; Temp Max (degC) (none) -> 125; Temp Min (degC) (none) -> -55; Temp Source (none) -> Legacy schematic field; primary-source verification pending; Temp Status (none) -> Inherited rating; system requirement pending
- R180, R181: Assembly (none) -> FIT; BOM Status (none) -> PART IDENTIFIED; sourcing/footprint review pending; Footprint Status (none) -> Assigned; drawing/pad verification pending; Function (none) -> Precision thermistor divider resistor; JLCPCB Library (none) -> UNVERIFIED; JLCPCB Status (none) -> LCSC exact match; JLC assembly availability unverified; LCSC (none) -> C110775; MPN (none) -> RT0805BRD0710KL; Manufacturer (none) -> Yageo; Operating Temperature (none) -> -55 to +155 C; Power (none) -> 0.125 W at 70 C; Supplier Data Checked (none) -> 2026-10-03; Supplier Source (none) -> https://lcsc.com/product-detail/Chip-Resistor-Surface-Mount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; TCR (none) -> 25 ppm/C; Temp Basis (none) -> Operating; power derates above 70 C; Temp Checked (none) -> 2026-10-03; Temp Max (degC) (none) -> 155; Temp Min (degC) (none) -> -55; Temp Source (none) -> https://www.yageogroup.com/component-documentation/download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; Temp Status (none) -> Manufacturer rating recorded; system requirement pending; Tolerance (none) -> 0.1%; Voltage (none) -> 150 V maximum working
- R182, R183: Assembly (none) -> FIT; BOM Status (none) -> PART IDENTIFIED; sourcing/footprint review pending; Footprint Status (none) -> Assigned; drawing/pad verification pending; Function (none) -> Resistor; JLCPCB Status (none) -> Historical ID; recheck exact part and assembly availability; LCSC (none) -> C95781; MPN (none) -> RC0805FR-071KL; Manufacturer (none) -> Yageo; Operating Temperature (none) -> -55 to +155 C; Supplier Data Checked (none) -> UNDATED legacy record; Supplier Source (none) -> Legacy schematic record; exact supplier listing verificatio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; Temp Basis (none) -> Legacy rating; ambient/junction basis unverified; Temp Max (degC) (none) -> 155; Temp Min (degC) (none) -> -55; Temp Source (none) -> Legacy schematic field; primary-source verification pending; Temp Status (none) -> Inherited rating; system requirement pending
- R65, R66, R67, R68: Assembly (none) -> FIT; BOM Status (none) -> PART IDENTIFIED; sourcing/footprint review pending; Footprint Status (none) -> Assigned; drawing/pad verification pending; Function (none) -> Resistor; JLCPCB Status (none) -> Historical ID; recheck exact part and assembly availability; MPN (none) -> RC0805FR-074K7L; Supplier Data Checked (none) -> UNDATED legacy record; Supplier Source (none) -> Legacy schematic record; exact supplier listing verificatio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; Temp Basis (none) -> Legacy rating; ambient/junction basis unverified; Temp Max (degC) (none) -> 155; Temp Min (degC) (none) -> -55; Temp Source (none) -> Legacy schematic field; primary-source verification pending; Temp Status (none) -> Inherited rating; system requirement pending
- TH1, TH2: Assembly (none) -> FIT; BOM Status (none) -> PART IDENTIFIED; sourcing/footprint review pending; Footprint Status (none) -> Assigned; drawing/pad verification pending; Function (none) -> Onboard 10 kohm NTC temperature sensor, 1206; Height (none) -> 1.30 mm max; JLCPCB Library (none) -> UNVERIFIED; JLCPCB Status (none) -> LCSC exact match; JLC assembly availability unverified; LCSC (none) -> C3152964; MPN (none) -> B57621C5103J062; Manufacturer (none) -> TDK; Operating Temperature (none) -> -55 to +125 C; Supplier Data Checked (none) -> 2026-10-03; Supplier Source (none) -> https://www.lcsc.com/product-detail/ntc-thermistors_tdk-b57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; Temp Basis (none) -> Category temperatures from climatic category 55/125/21; acc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; Temp Checked (none) -> 2026-10-03; Temp Max (degC) (none) -> 125; Temp Min (degC) (none) -> -55; Temp Source (none) -> https://www.tdk-electronics.tdk.com/en/530414/products/prod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; Temp Status (none) -> Manufacturer rating recorded; system requirement pending; Tolerance (none) -> 5% at 25 C
- U21: Assembly (none) -> FIT; BOM Status (none) -> PART IDENTIFIED; sourcing/footprint review pending; Footprint Status (none) -> Assigned; drawing/pad verification pending; Function (none) -> ADS1115BQDGSRQ1; JLCPCB Status (none) -> Historical ID; recheck exact part and assembly availability; MPN (none) -> ADS1115BQDGSRQ1; Supplier Data Checked (none) -> UNDATED legacy record; Supplier Source (none) -> Legacy schematic record; exact supplier listing verificatio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; Temp Basis (none) -> Legacy rating; ambient/junction basis unverified; Temp Max (degC) (none) -> 125; Temp Min (degC) (none) -> -40; Temp Source (none) -> Legacy schematic field; primary-source verification pending; Temp Status (none) -> Inherited rating; system requirement pending
- U24: Assembly (none) -> FIT; BOM Status (none) -> PART IDENTIFIED; sourcing/footprint review pending; Footprint Status (none) -> Assigned; drawing/pad verification pending; Function (none) -> ISO1540DR; JLCPCB Status (none) -> Historical ID; recheck exact part and assembly availability; MPN (none) -> ISO1540DR; Supplier Data Checked (none) -> UNDATED legacy record; Supplier Source (none) -> Legacy schematic record; exact supplier listing verificatio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; Temp Basis (none) -> Legacy rating; ambient/junction basis unverified; Temp Max (degC) (none) -> 125; Temp Min (degC) (none) -> -40; Temp Source (none) -> Legacy schematic field; primary-source verification pending; Temp Status (none) -> Inherited rating; system requirement pending
