File: Brakes.kicad_sch (KiCad schematic)
At the start: 49 parts, among them IC1 TPS1H100BQPWPRQ1, IC2 TPS1H100BQPWPRQ1, J7 DE9_Socket_MountingHoles, U2 ISO6762FQDWRQ1, U5 TPD2E2U06QDBZRQ1

Commit message: Redesign schematic for dual motor encoders
Parts:
- TP10: value RH_BRAKE_COIL -> STAR_BRAKE_COIL
- TP6: value +6.5V_ENC_L -> +6.5V_ENC_PORT
- TP7: value +6.5V_ENC_R -> +6.5V_ENC_STAR
- TP9: value LH_BRAKE_COIL -> PORT_BRAKE_COIL
Connections:
- net +6.5V_ENC_L renamed +6.5V_ENC_PORT
- net +6.5V_ENC_R renamed +6.5V_ENC_STAR
- net LH_BRAKE_COIL renamed PORT_BRAKE_COIL
- net LH_BRAKE_CURR renamed PORT_BRAKE_CURR
- net LH_BRAKE_RELEASE_CMD renamed PORT_BRAKE_RELEASE_CMD
- net RH_BRAKE_COIL renamed STAR_BRAKE_COIL
- net RH_BRAKE_CURR renamed STAR_BRAKE_CURR
- net RH_BRAKE_RELEASE_CMD renamed STAR_BRAKE_RELEASE_CMD
Other:
- note added: "Digital isolator"
- note added: "Port brake high-side switch"
- note added: "Signal ESD protection"
- note added: "Star brake high-side switch"
Changed lines of the file:
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@@
 	(title_block
 		(title "Elevation Control_Gigabit")
-		(date "2026-09-01")
-		(rev "Sep_2026_V1")
+		(date "2026-10-03")
+		(rev "P3 REVIEW")
 		(company "Starspec")
 		(comment 4 "Mauro M. Coutinho")
@@
 		)
 	)
+	(text "Port brake high-side switch"
+		(exclude_from_sim no)
+		(at 193.04 30.48 0)
+		(effects
+			(font
+				(size 1.27 1.27)
+			)
+		)
+	)
 	(text "0V going \nto switch"
 		(exclude_from_sim no)
@@
 		)
 	)
+	(text "Signal ESD protection"
+		(exclude_from_sim no)
+		(at 187.96 168.91 0)
+		(effects
+			(font
+				(size 1.27 1.27)
+			)
+		)
+	)
+	(text "Digital isolator"
+		(exclude_from_sim no)
+		(at 96.52 30.48 0)
+		(effects
+			(font
+				(size 1.27 1.27)
+			)
+		)
+	)
 	(text "The onsemi MBR3100RLG, a 3 A, 100 V \naxial Schottky diode should be \ninstalled on the brake harness!!\n\n"
 		(exclude_from_sim no)
@@
 		)
 	)
+	(text "Star brake high-side switch"
+		(exclude_from_sim no)
+		(at 191.77 97.79 0)
+		(effects
+			(font
+				(size 1.27 1.27)
+			)
+		)
+	)
 	(text "I_LIMIT = (1.233Ã—2000) / RCL\n	â€‹\nRCL (R1) = 1.00 kÎ©, 1%\nNominal current limit â‰ˆ 2.47 A"
 		(exclude_from_sim no)
@@
 		)
 	)
-	(global_label "RH_BRAKE_COIL"
+	(global_label "STAR_BRAKE_COIL"
 		(shape input)
 		(at 172.72 119.38 180)
@@
 		)
 	)
-	(global_label "RH_BRAKE_COIL"
+	(global_label "STAR_BRAKE_COIL"
 		(shape input)
 		(at 67.31 176.53 180)
@@
 		)
 	)
-	(global_label "LH_BRAKE_COIL"
+	(global_label "PORT_BRAKE_COIL"
 		(shape input)
 		(at 67.31 161.29 180)
@@
 		)
 	)
-	(global_label "+6.5V_ENC_L"
+	(global_label "+6.5V_ENC_PORT"
 		(shape input)
 		(at 300.99 83.82 0)
@@
 		)
 	)
-	(global_label "LH_BRAKE_COIL"
+	(global_label "PORT_BRAKE_COIL"
 		(shape input)
 		(at 300.99 121.92 0)
@@
 		)
 	)
-	(global_label "+6.5V_ENC_R"
+	(global_label "+6.5V_ENC_STAR"
 		(shape input)
 		(at 300.99 96.52 0)
@@
 		)
 	)
-	(global_label "RH_BRAKE_COIL"
+	(global_label "STAR_BRAKE_COIL"
 		(shape input)
 		(at 300.99 134.62 0)
@@
 		)
 	)
-	(global_label "LH_BRAKE_COIL"
+	(global_label "PORT_BRAKE_COIL"
 		(shape input)
 		(at 173.99 52.07 180)
@@
 		)
 	)
-	(hierarchical_label "RH_BRAKE_RELEASE_CMD"
+	(hierarchical_label "STAR_BRAKE_RELEASE_CMD"
 		(shape input)
 		(at 35.56 49.53 270)
@@
 		)
 	)
-	(hierarchical_label "LH_BRAKE_RELEASE_CMD"
+	(hierarchical_label "PORT_BRAKE_RELEASE_CMD"
 		(shape input)
 		(at 21.59 46.99 270)
@@
 		)
 	)
-	(hierarchical_label "LH_BRAKE_CURR"
+	(hierarchical_label "PORT_BRAKE_CURR"
 		(shape output)
 		(at 261.62 41.91 0)
@@
 		)
 	)
-	(hierarchical_label "RH_BRAKE_CURR"
+	(hierarchical_label "STAR_BRAKE_CURR"
 		(shape output)
 		(at 261.62 109.22 0)
@@
 			)
 		)
-		(property "Value" "+6.5V_ENC_L"
+		(property "Value" "+6.5V_ENC_PORT"
 			(at 285.75 85.62 0)
 			(effects
@@
 			)
 		)
-		(property "Value" "+6.5V_ENC_R"
+		(property "Value" "+6.5V_ENC_STAR"
 			(at 285.75 98.32 0)
 			(effects
@@
 			)
 		)
-		(property "Value" "RH_BRAKE_COIL"
+		(property "Value" "STAR_BRAKE_COIL"
 			(at 285.75 136.42 0)
 			(effects
@@
 			)
 		)
-		(property "Value" "LH_BRAKE_COIL"
+		(property "Value" "PORT_BRAKE_COIL"
 			(at 285.75 123.72 0)
 			(effects

Commit message: Preserve P5 equal-size placement, controller stack and native BOM
Parts:
- C22, C27, C36, C45: Assembly (none) -> FIT; BOM Status (none) -> PART IDENTIFIED; sourcing/footprint review pending; Footprint Status (none) -> Assigned; drawing/pad verification pending; Function (none) -> Unpolarized capacitor; JLCPCB Status (none) -> Historical ID; recheck exact part and assembly availability; MPN (none) -> CL21B474KBFNNNE; Supplier Data Checked (none) -> UNDATED legacy record; Supplier Source (none) -> Legacy schematic record; exact supplier listing verificatio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; Temp Basis (none) -> Legacy rating; ambient/junction basis unverified; Temp Max (degC) (none) -> 125; Temp Min (degC) (none) -> -55; Temp Source (none) -> Legacy schematic field; primary-source verification pending; Temp Status (none) -> Inherited rating; system requirement pending
- C24, C25, C34, C43: Assembly (none) -> FIT; BOM Status (none) -> PART IDENTIFIED; sourcing/footprint review pending; Footprint Status (none) -> Assigned; drawing/pad verification pending; Function (none) -> Unpolarized capacitor; JLCPCB Status (none) -> Historical ID; recheck exact part and assembly availability; MPN (none) -> CL21B104KCFNNNE; Supplier Data Checked (none) -> UNDATED legacy record; Supplier Source (none) -> Legacy schematic record; exact supplier listing verificatio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; Temp Basis (none) -> Legacy rating; ambient/junction basis unverified; Temp Max (degC) (none) -> 125; Temp Min (degC) (none) -> -55; Temp Source (none) -> Legacy schematic field; primary-source verification pending; Temp Status (none) -> Inherited rating; system requirement pending
- C26, C4: Assembly (none) -> FIT; BOM Status (none) -> PART IDENTIFIED; sourcing/footprint review pending; Footprint Status (none) -> Assigned; drawing/pad verification pending; Function (none) -> Unpolarized capacitor; JLCPCB Status (none) -> Historical ID; recheck exact part and assembly availability; MPN (none) -> CL31B105KCHNNNE; Supplier Data Checked (none) -> UNDATED legacy record; Supplier Source (none) -> Legacy schematic record; exact supplier listing verificatio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; Temp Basis (none) -> Legacy rating; ambient/junction basis unverified; Temp Max (degC) (none) -> 125; Temp Min (degC) (none) -> -55; Temp Source (none) -> Legacy schematic field; primary-source verification pending; Temp Status (none) -> Inherited rating; system requirement pending
- C28, C33, C39, C41: Assembly (none) -> FIT; BOM Status (none) -> PART IDENTIFIED; sourcing/footprint review pending; Footprint Status (none) -> Assigned; drawing/pad verification pending; Function (none) -> Unpolarized capacitor; JLCPCB Status (none) -> Historical ID; recheck exact part and assembly availability; MPN (none) -> FS55X106K101EHG; Supplier Data Checked (none) -> UNDATED legacy record; Supplier Source (none) -> Legacy schematic record; exact supplier listing verificatio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; Temp Basis (none) -> Legacy rating; ambient/junction basis unverified; Temp Max (degC) (none) -> 125; Temp Min (degC) (none) -> -55; Temp Source (none) -> Legacy schematic field; primary-source verification pending; Temp Status (none) -> Inherited rating; system requirement pending
- D10, D11: Assembly (none) -> DNP - not purchased; BOM Status (none) -> DNP; Footprint Status (none) -> Assigned; drawing/pad verification pending; Function (none) -> STPS3H100U; JLCPCB Status (none) -> No verified JLCPCB ID; source or consign; LCSC (none) -> UNVERIFIED; MPN (none) -> STPS3H100U; Operating Temperature See datasheet -> NOT SELECTED - DNP; Supplier Data Checked (none) -> UNDATED legacy record; Supplier Source (none) -> Legacy schematic record; exact supplier listing verificatio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; Temp Basis (none) -> Primary-source verification pending; Temp Max (degC) (none) -> N/A; Temp Min (degC) (none) -> N/A; Temp Status (none) -> NOT_EVALUATED_DNP
- F1, F2: Assembly (none) -> FIT; BOM Review (none) -> Existing brake fuse retained. Resolve against user preferen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; BOM Status (none) -> REVIEW: legacy brake fuse versus no-fuse preference; Footprint Status (none) -> Assigned; drawing/pad verification pending; Function (none) -> Fuse; JLCPCB Status (none) -> Historical ID; recheck exact part and assembly availability; MPN (none) -> 0466002.NRHF; Supplier Data Checked (none) -> UNDATED legacy record; Supplier Source (none) -> Legacy schematic record; exact supplier listing verificatio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; Temp Basis (none) -> Legacy rating; ambient/junction basis unverified; Temp Max (degC) (none) -> 90; Temp Min (degC) (none) -> -55; Temp Source (none) -> Legacy schematic field; primary-source verification pending; Temp Status (none) -> Inherited rating; system requirement pending
- IC1, IC2: Assembly (none) -> FIT; BOM Status (none) -> PART IDENTIFIED; sourcing/footprint review pending; Footprint Status (none) -> Assigned; drawing/pad verification pending; Function (none) -> Power Switch ICs - Power Distribution 40V/100mOhm Sngl Chn; JLCPCB Status (none) -> Historical ID; recheck exact part and assembly availability; MPN (none) -> TPS1H100BQPWPRQ1; Supplier Data Checked (none) -> UNDATED legacy record; Supplier Source (none) -> Legacy schematic record; exact supplier listing verificatio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; Temp Basis (none) -> Legacy rating; ambient/junction basis unverified; Temp Max (degC) (none) -> 125; Temp Min (degC) (none) -> -40; Temp Source (none) -> Legacy schematic field; primary-source verification pending; Temp Status (none) -> Inherited rating; system requirement pending
- J7: Assembly (none) -> FIT; BOM Review (none) -> Same MPN as existing DE9 connectors. Verify exact pin grid,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; BOM Status (none) -> PART IDENTIFIED; sourcing/footprint review pending; Footprint Status (none) -> REVIEW: compare exact TE drawing to generic KiCad footprint; Function (none) -> DE9 female right-angle PCB connector; JLCPCB Library (none) -> UNVERIFIED; JLCPCB Status (none) -> LCSC exact match; JLC assembly availability unverified; MPN (none) -> 5747844-4; Supplier Data Checked (none) -> 2026-10-03; Supplier Source (none) -> https://www.lcsc.com/de/product-detail/C305941.html; Temp Basis (none) -> Operating; Temp Checked (none) -> 2026-10-03; Temp Max (degC) (none) -> 105; Temp Min (degC) (none) -> -55; Temp Source (none) -> https://www.te.com/en/product-5747844-4.html; Temp Status (none) -> Manufacturer rating recorded; system requirement pending
- R1, R21: Assembly (none) -> FIT; BOM Status (none) -> PART IDENTIFIED; sourcing/footprint review pending; Footprint Status (none) -> Assigned; drawing/pad verification pending; Function (none) -> Resistor; JLCPCB Status (none) -> Historical ID; recheck exact part and assembly availability; MPN (none) -> RC0805FR-071KL; Supplier Data Checked (none) -> UNDATED legacy record; Supplier Source (none) -> Legacy schematic record; exact supplier listing verificatio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; Temp Basis (none) -> Legacy rating; ambient/junction basis unverified; Temp Max (degC) (none) -> 155; Temp Min (degC) (none) -> -55; Temp Source (none) -> Legacy schematic field; primary-source verification pending; Temp Status (none) -> Inherited rating; system requirement pending
- R11, R23, R24, R26, R43, R44, R9: Assembly (none) -> FIT; BOM Status (none) -> PART IDENTIFIED; sourcing/footprint review pending; Footprint Status (none) -> Assigned; drawing/pad verification pending; Function (none) -> Resistor; JLCPCB Status (none) -> Historical ID; recheck exact part and assembly availability; MPN (none) -> RC0805FR-0747KL; Supplier Data Checked (none) -> UNDATED legacy record; Supplier Source (none) -> Legacy schematic record; exact supplier listing verificatio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; Temp Basis (none) -> Legacy rating; ambient/junction basis unverified; Temp Max (degC) (none) -> 155; Temp Min (degC) (none) -> -55; Temp Source (none) -> Legacy schematic field; primary-source verification pending; Temp Status (none) -> Inherited rating; system requirement pending
- R18, R25, R5: Assembly (none) -> FIT; BOM Status (none) -> PART IDENTIFIED; sourcing/footprint review pending; Footprint Status (none) -> Assigned; drawing/pad verification pending; Function (none) -> Resistor; JLCPCB Status (none) -> Historical ID; recheck exact part and assembly availability; MPN (none) -> RC0805FR-0710KL; Supplier Data Checked (none) -> UNDATED legacy record; Supplier Source (none) -> Legacy schematic record; exact supplier listing verificatio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; Temp Basis (none) -> Legacy rating; ambient/junction basis unverified; Temp Max (degC) (none) -> 155; Temp Min (degC) (none) -> -55; Temp Source (none) -> Legacy schematic field; primary-source verification pending; Temp Status (none) -> Inherited rating; system requirement pending
- R19, R20: Assembly (none) -> FIT; BOM Status (none) -> PART IDENTIFIED; sourcing/footprint review pending; Footprint Status (none) -> Assigned; drawing/pad verification pending; Function (none) -> Resistor; JLCPCB Status (none) -> Historical ID; recheck exact part and assembly availability; MPN (none) -> RC0805FR-07430RL; Supplier Data Checked (none) -> UNDATED legacy record; Supplier Source (none) -> Legacy schematic record; exact supplier listing verificatio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; Temp Basis (none) -> Legacy rating; ambient/junction basis unverified; Temp Max (degC) (none) -> 155; Temp Min (degC) (none) -> -55; Temp Source (none) -> Legacy schematic field; primary-source verification pending; Temp Status (none) -> Inherited rating; system requirement pending
- R22, R3: Assembly (none) -> FIT; BOM Status (none) -> PART IDENTIFIED; sourcing/footprint review pending; Footprint Status (none) -> Assigned; drawing/pad verification pending; Function (none) -> Resistor; JLCPCB Status (none) -> Historical ID; recheck exact part and assembly availability; MPN (none) -> RC0805FR-07560RL; Supplier Data Checked (none) -> UNDATED legacy record; Supplier Source (none) -> Legacy schematic record; exact supplier listing verificatio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; Temp Basis (none) -> Legacy rating; ambient/junction basis unverified; Temp Max (degC) (none) -> 155; Temp Min (degC) (none) -> -55; Temp Source (none) -> Legacy schematic field; primary-source verification pending; Temp Status (none) -> Inherited rating; system requirement pending
- TP1, TP10, TP2, TP3, TP4, TP5, TP6, TP7, TP8, TP9: Assembly (none) -> PCB feature - no purchased component; BOM Status (none) -> PCB FEATURE; Function (none) -> PCB test pad; JLCPCB Status (none) -> N/A; LCSC (none) -> N/A; MPN (none) -> N/A; Manufacturer (none) -> N/A; Operating Temperature (none) -> N/A; Temp Basis (none) -> PCB feature; Temp Max (degC) (none) -> N/A; Temp Min (degC) (none) -> N/A; Temp Status (none) -> N/A
- U2: Assembly (none) -> FIT; BOM Status (none) -> PART IDENTIFIED; sourcing/footprint review pending; Footprint Status (none) -> Assigned; drawing/pad verification pending; Function (none) -> ISO6762FQDWRQ1; JLCPCB Status (none) -> Historical ID; recheck exact part and assembly availability; MPN (none) -> ISO6762FQDWRQ1; Supplier Data Checked (none) -> UNDATED legacy record; Supplier Source (none) -> Legacy schematic record; exact supplier listing verificatio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; Temp Basis (none) -> Legacy rating; ambient/junction basis unverified; Temp Max (degC) (none) -> 125; Temp Min (degC) (none) -> -40; Temp Source (none) -> Legacy schematic field; primary-source verification pending; Temp Status (none) -> Inherited rating; system requirement pending
- U5: Assembly (none) -> FIT; BOM Status (none) -> PART IDENTIFIED; sourcing/footprint review pending; Footprint Status (none) -> Assigned; drawing/pad verification pending; Function (none) -> Automotive Dual-Channel High-Speed ESD Protection Device; JLCPCB Status (none) -> Historical ID; recheck exact part and assembly availability; MPN (none) -> TPD2E2U06QDBZRQ1; Supplier Data Checked (none) -> UNDATED legacy record; Supplier Source (none) -> Legacy schematic record; exact supplier listing verificatio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; Temp Basis (none) -> Legacy rating; ambient/junction basis unverified; Temp Max (degC) (none) -> 125; Temp Min (degC) (none) -> -40; Temp Source (none) -> Legacy schematic field; primary-source verification pending; Temp Status (none) -> Inherited rating; system requirement pending

Commit message: Build P6 80x130 stack with redistributed SSI and stepper interfaces
Other:
- note added: "I_LIMIT = (1.233Ã—2000) / RCL tâ€‹ RCL (R1) = 1.00 kÎ©, 1% Nominal current limit â‰ˆ 2.47 A"
- note removed: "I_LIMIT = (1.233Ã—2000) / RCL â€‹ RCL (R1) = 1.00 kÎ©, 1% Nominal current limit â‰ˆ 2.47 A"
