File: DC_DC_Step_Down.kicad_sch (KiCad schematic)
At the start: 59 parts, among them J1 1827884, U14 R05CTE05S-R, U23 TPS7A2450DBVR, U25 TPS7A2450DBVR

Commit message: Redesign schematic for dual motor encoders
Connections:
- net +5V_ENC_L renamed +5V_ENC_PORT
- net +5V_ENC_R renamed +5V_ENC_STAR
- net +6.5V_ENC_L renamed +6.5V_ENC_PORT
- net +6.5V_ENC_R renamed +6.5V_ENC_STAR
Other:
- note added: "5 V brake supply"
- note added: "5 V field supply"
- note added: "5 V linear regulator"
- note added: "6.5 V Port SSI supply"
- note added: "6.5 V Star SSI supply"
- note added: "Common-mode filter"
- note added: "Isolated 5 V CAN supply"
- note added: "Isolated 5 V MCU supply"
Changed lines of the file:
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@@
 	(title_block
 		(title "Elevation Control_Gigabit")
-		(date "2026-09-01")
-		(rev "Sep_2026_V1")
+		(date "2026-10-03")
+		(rev "P3 REVIEW")
 		(company "Starspec")
 		(comment 4 "Mauro M. Coutinho")
 	)
+	(text "5 V linear regulator"
+		(exclude_from_sim no)
+		(at 175.26 182.88 0)
+		(effects
+			(font
+				(size 1.27 1.27)
+			)
+		)
+	)
+	(text "5 V linear regulator"
+		(exclude_from_sim no)
+		(at 176.53 226.06 0)
+		(effects
+			(font
+				(size 1.27 1.27)
+			)
+		)
+	)
 	(text "External supply / return entry at J1 (ERC source declarations)"
 		(exclude_from_sim no)
@@
 		)
 	)
+	(text "5 V field supply"
+		(exclude_from_sim no)
+		(at 76.2 92.71 0)
+		(effects
+			(font
+				(size 1.27 1.27)
+			)
+		)
+	)
+	(text "6.5 V Star SSI supply"
+		(exclude_from_sim no)
+		(at 66.04 214.63 0)
+		(effects
+			(font
+				(size 1.27 1.27)
+			)
+		)
+	)
+	(text "6.5 V Port SSI supply"
+		(exclude_from_sim no)
+		(at 67.31 168.91 0)
+		(effects
+			(font
+				(size 1.27 1.27)
+			)
+		)
+	)
+	(text "Isolated 5 V MCU supply"
+		(exclude_from_sim no)
+		(at 140.97 33.02 0)
+		(effects
+			(font
+				(size 1.27 1.27)
+			)
+		)
+	)
+	(text "Common-mode filter"
+		(exclude_from_sim no)
+		(at 81.28 33.02 0)
+		(effects
+			(font
+				(size 1.27 1.27)
+			)
+		)
+	)
+	(text "5 V brake supply"
+		(exclude_from_sim no)
+		(at 356.87 22.86 0)
+		(effects
+			(font
+				(size 1.27 1.27)
+			)
+		)
+	)
 	(text "DNC --"
 		(exclude_from_sim no)
@@
 		)
 	)
+	(text "Isolated 5 V CAN supply"
+		(exclude_from_sim no)
+		(at 279.4 101.6 0)
+		(effects
+			(font
+				(size 1.27 1.27)
+			)
+		)
+	)
 	(text "173010575 (1000 mAmp)\n173950575 (500 mAmp)"
 		(exclude_from_sim no)
@@
 	(wire
 		(pts
-			(xy 269.24 78.74) (xy 279.4 78.74)
-		)
-		(stroke
-			(width 0)
-			(type default)
-		)
-	)
-	(wire
-		(pts
 			(xy 81.28 250.19) (xy 92.71 250.19)
 		)
@@
 	(wire
 		(pts
+			(xy 269.24 76.2) (xy 269.24 78.74)
+		)
+		(stroke
+			(width 0)
+			(type default)
+		)
+	)
+	(wire
+		(pts
 			(xy 66.04 207.01) (xy 66.04 205.74)
 		)
@@
 	(wire
 		(pts
+			(xy 330.2 77.47) (xy 330.2 78.74)
+		)
+		(stroke
+			(width 0)
+			(type default)
+		)
+	)
+	(wire
+		(pts
 			(xy 308.61 125.73) (xy 308.61 128.27)
 		)
@@
 	(wire
 		(pts
-			(xy 330.2 78.74) (xy 340.36 78.74)
-		)
-		(stroke
-			(width 0)
-			(type default)
-		)
-	)
-	(wire
-		(pts
 			(xy 119.38 31.75) (xy 119.38 44.45)
 		)
@@
 	)
 	(symbol
-		(lib_id "Power_Custom:+5V_ENC_R")
+		(lib_id "Power_Custom:+5V_ENC_STAR")
 		(at 222.25 236.22 0)
 		(unit 1)
@@
 			)
 		)
-		(property "Value" "+5V_ENC_R"
+		(property "Value" "+5V_ENC_STAR"
 			(at 222.25 231.14 0)
 			(effects
@@
 	(symbol
 		(lib_id "power:PWR_FLAG")
-		(at 279.4 78.74 0)
+		(at 269.24 76.2 0)
 		(unit 1)
 		(exclude_from_sim no)
@@
 		(dnp no)
 		(property "Reference" "#FLG04"
-			(at 279.4 78.74 0)
+			(at 269.24 76.2 0)
 			(effects
 				(font
@@
 		)
 		(property "Value" "PWR_FLAG"
-			(at 279.4 73.66 0)
+			(at 269.24 71.12 0)
 			(effects
 				(font
@@
 		)
 		(property "Footprint" ""
-			(at 279.4 78.74 0)
+			(at 269.24 76.2 0)
 			(effects
 				(font
@@
 		)
 		(property "Datasheet" "~"
-			(at 279.4 78.74 0)
+			(at 269.24 76.2 0)
 			(effects
 				(font
@@
 		)
 		(property "Description" ""
-			(at 279.4 78.74 0)
+			(at 269.24 76.2 0)
 			(effects
 				(font
@@
 	)
 	(symbol
-		(lib_id "Power_Custom:6.5V_ENC_L")
+		(lib_id "Power_Custom:6.5V_ENC_PORT")
 		(at 144.78 236.22 0)
 		(unit 1)
@@
 			)
 		)
-		(property "Value" "+6.5V_ENC_R"
+		(property "Value" "+6.5V_ENC_STAR"
 			(at 144.78 231.14 0)
 			(effects
@@
 	(symbol
 		(lib_id "power:PWR_FLAG")
-		(at 340.36 78.74 0)
+		(at 330.2 77.47 0)
 		(unit 1)
 		(exclude_from_sim no)
@@
 		(dnp no)
 		(property "Reference" "#FLG06"
-			(at 340.36 78.74 0)
+			(at 330.2 77.47 0)
 			(effects
 				(font
@@
 		)
 		(property "Value" "PWR_FLAG"
-			(at 340.36 73.66 0)
+			(at 330.2 72.39 0)
 			(effects
 				(font
@@
 		)
 		(property "Footprint" ""
-			(at 340.36 78.74 0)
+			(at 330.2 77.47 0)
 			(effects
 				(font
@@
 		)
 		(property "Datasheet" "~"
-			(at 340.36 78.74 0)
+			(at 330.2 77.47 0)
 			(effects
 				(font
@@
 		)
 		(property "Description" ""
-			(at 340.36 78.74 0)
+			(at 330.2 77.47 0)
 			(effects
 				(font
@@
 	)
 	(symbol
-		(lib_id "Power_Custom:6.5V_ENC_L")
+		(lib_id "Power_Custom:6.5V_ENC_PORT")
 		(at 182.88 260.35 0)
 		(unit 1)
@@
 			)
 		)
-		(property "Value" "+6.5V_ENC_R"
+		(property "Value" "+6.5V_ENC_STAR"
 			(at 182.88 255.27 0)
 			(effects
@@
 	)
 	(symbol
-		(lib_id "Power_Custom:6.5V_ENC_L")
+		(lib_id "Power_Custom:6.5V_ENC_PORT")
 		(at 144.78 193.04 0)
 		(unit 1)
@@
 			)
 		)
-		(property "Value" "+6.5V_ENC_L"
+		(property "Value" "+6.5V_ENC_PORT"
 			(at 144.78 187.96 0)
 			(effects
@@
 	)
 	(symbol
-		(lib_id "Power_Custom:6.5V_ENC_L")
+		(lib_id "Power_Custom:6.5V_ENC_PORT")
 		(at 181.61 214.63 0)
 		(unit 1)
@@
 			)
 		)
-		(property "Value" "+6.5V_ENC_L"
+		(property "Value" "+6.5V_ENC_PORT"
 			(at 181.61 209.55 0)
 			(effects
@@
 	)
 	(symbol
-		(lib_id "Power_Custom:+5V_ENC_L")
+		(lib_id "Power_Custom:+5V_ENC_PORT")
 		(at 223.52 194.31 0)
 		(unit 1)
@@
 			)
 		)
-		(property "Value" "+5V_ENC_L"
+		(property "Value" "+5V_ENC_PORT"
 			(at 223.52 189.23 0)
 			(effects

Commit message: Preserve P5 equal-size placement, controller stack and native BOM
Parts:
- C1, C101, C103, C20, C35, C46, C49, C55, C75, C77, C8, C80, C83, C85, C92, C94: Assembly (none) -> FIT; BOM Status (none) -> PART IDENTIFIED; sourcing/footprint review pending; Footprint Status (none) -> Assigned; drawing/pad verification pending; Function (none) -> Unpolarized capacitor; JLCPCB Status (none) -> Historical ID; recheck exact part and assembly availability; MPN (none) -> CL21B104KCFNNNE; Supplier Data Checked (none) -> UNDATED legacy record; Supplier Source (none) -> Legacy schematic record; exact supplier listing verificatio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; Temp Basis (none) -> Legacy rating; ambient/junction basis unverified; Temp Max (degC) (none) -> 125; Temp Min (degC) (none) -> -55; Temp Source (none) -> Legacy schematic field; primary-source verification pending; Temp Status (none) -> Inherited rating; system requirement pending
- C10, C11, C12, C21, C47, C48, C5, C73, C74, C81, C82: Assembly (none) -> FIT; BOM Status (none) -> PART IDENTIFIED; sourcing/footprint review pending; Footprint Status (none) -> Assigned; drawing/pad verification pending; Function (none) -> Unpolarized capacitor; JLCPCB Status (none) -> Historical ID; recheck exact part and assembly availability; MPN (none) -> FS55X106K101EHG; Supplier Data Checked (none) -> UNDATED legacy record; Supplier Source (none) -> Legacy schematic record; exact supplier listing verificatio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; Temp Basis (none) -> Legacy rating; ambient/junction basis unverified; Temp Max (degC) (none) -> 125; Temp Min (degC) (none) -> -55; Temp Source (none) -> Legacy schematic field; primary-source verification pending; Temp Status (none) -> Inherited rating; system requirement pending
- C100, C102, C13, C14, C44, C54, C7, C79: Assembly (none) -> FIT; BOM Status (none) -> PART IDENTIFIED; sourcing/footprint review pending; Footprint Status (none) -> Assigned; drawing/pad verification pending; Function (none) -> Unpolarized capacitor; JLCPCB Status (none) -> Historical ID; recheck exact part and assembly availability; MPN (none) -> CL32B475KCVZNWE; Supplier Data Checked (none) -> UNDATED legacy record; Supplier Source (none) -> Legacy schematic record; exact supplier listing verificatio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; Temp Basis (none) -> Legacy rating; ambient/junction basis unverified; Temp Max (degC) (none) -> 125; Temp Min (degC) (none) -> -55; Temp Source (none) -> Legacy schematic field; primary-source verification pending; Temp Status (none) -> Inherited rating; system requirement pending
- C16: Assembly (none) -> DNP - not purchased; BOM Status (none) -> DNP; Footprint Status (none) -> Assigned; drawing/pad verification pending; Function (none) -> Unpolarized capacitor; JLCPCB Status (none) -> Historical ID; recheck exact part and assembly availability; MPN (none) -> GA355DR7GF472KW01L; Supplier Data Checked (none) -> UNDATED legacy record; Supplier Source (none) -> Legacy schematic record; exact supplier listing verificatio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; Temp Basis (none) -> Legacy rating; ambient/junction basis unverified; Temp Max (degC) (none) -> 125; Temp Min (degC) (none) -> -55; Temp Source (none) -> Legacy schematic field; primary-source verification pending; Temp Status (none) -> Inherited rating; system requirement pending
- C23, C50, C61, C76, C78, C84, C86, C93, C95: Assembly (none) -> FIT; BOM Status (none) -> PART IDENTIFIED; sourcing/footprint review pending; Footprint Status (none) -> Assigned; drawing/pad verification pending; Function (none) -> Unpolarized capacitor; JLCPCB Status (none) -> Historical ID; recheck exact part and assembly availability; MPN (none) -> CL32B106KBJNFNE; Supplier Data Checked (none) -> UNDATED legacy record; Supplier Source (none) -> Legacy schematic record; exact supplier listing verificatio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; Temp Basis (none) -> Legacy rating; ambient/junction basis unverified; Temp Max (degC) (none) -> 125; Temp Min (degC) (none) -> -55; Temp Source (none) -> Legacy schematic field; primary-source verification pending; Temp Status (none) -> Inherited rating; system requirement pending
- FB1, FB2, FB3: Assembly (none) -> FIT; BOM Status (none) -> PART IDENTIFIED; sourcing/footprint review pending; Footprint Status (none) -> Assigned; drawing/pad verification pending; Function (none) -> Ferrite bead; JLCPCB Status (none) -> Historical ID; recheck exact part and assembly availability; MPN (none) -> MPZ2012S601ATD25; Supplier Data Checked (none) -> UNDATED legacy record; Supplier Source (none) -> Legacy schematic record; exact supplier listing verificatio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; Temp Basis (none) -> Legacy rating; ambient/junction basis unverified; Temp Max (degC) (none) -> 125; Temp Min (degC) (none) -> -55; Temp Source (none) -> Legacy schematic field; primary-source verification pending; Temp Status (none) -> Inherited rating; system requirement pending
- FL1: Assembly (none) -> FIT; BOM Review (none) -> Selected C0502 part uses a footprint named C0104; compare e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; BOM Status (none) -> REVIEW: legacy footprint name differs from MPN; Footprint Status (none) -> Assigned; drawing/pad verification pending; Function (none) -> Common Mode Filters / Chokes, |Z|=190 at 10MHz, L x W x T :; JLCPCB Status (none) -> Historical ID; recheck exact part and assembly availability; MPN (none) -> B82793C0502N201; Operating Temperature See datasheet -> -40 to +125 C; Supplier Data Checked (none) -> UNDATED legacy record; Supplier Source (none) -> Legacy schematic record; exact supplier listing verificatio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; Temp Basis (none) -> Operating; Temp Checked (none) -> 2026-10-03; Temp Max (degC) (none) -> 125; Temp Min (degC) (none) -> -40; Temp Source (none) -> https://product.tdk.com/en/search/emc/emc/cmf_cmc/info?part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; Temp Status (none) -> Manufacturer rating recorded; system requirement pending
- J1: Assembly (none) -> FIT; BOM Review (none) -> Manufacturer PDF specifies -40 to +100 C operation; confirm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; BOM Status (none) -> PART IDENTIFIED; sourcing/footprint review pending; Footprint Status (none) -> Assigned; drawing/pad verification pending; Function (none) -> 1827884; JLCPCB Status (none) -> No verified JLCPCB ID; source or consign; LCSC (none) -> UNVERIFIED; MPN (none) -> 1827884; Operating Temperature See datasheet -> -40 to +100 C (derated); Supplier Data Checked (none) -> UNDATED legacy record; Supplier Source (none) -> Legacy schematic record; exact supplier listing verificatio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; Temp Basis (none) -> Ambient operation with current derating; Temp Checked (none) -> 2026-10-03; Temp Max (degC) (none) -> 100; Temp Min (degC) (none) -> -40; Temp Source (none) -> https://www.phoenixcontact.com/gb/products/1827884/pdf; Temp Status (none) -> Manufacturer rating recorded; system requirement pending
- L1: Assembly (none) -> FIT; BOM Review (none) -> Confirm exact manufacturer dimensions and assembled height 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; BOM Status (none) -> PART IDENTIFIED; sourcing/footprint review pending; Footprint Status (none) -> Assigned; drawing/pad verification pending; Function (none) -> WE-PD SMT Shielded Power Inductor Size 1210; L = 33 H +/-20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; JLCPCB Status (none) -> Historical ID; recheck exact part and assembly availability; MPN (none) -> 7447709330; Operating Temperature See datasheet -> -40 to +125 C; Supplier Data Checked (none) -> UNDATED legacy record; Supplier Source (none) -> Legacy schematic record; exact supplier listing verificatio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; Temp Basis (none) -> Operating including self-heating; Temp Checked (none) -> 2026-10-03; Temp Max (degC) (none) -> 125; Temp Min (degC) (none) -> -40; Temp Source (none) -> https://www.we-online.com/components/products/datasheet/744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; Temp Status (none) -> Manufacturer rating recorded; system requirement pending
- PS1: Assembly (none) -> FIT; BOM Status (none) -> PART IDENTIFIED; sourcing/footprint review pending; Footprint Status (none) -> Assigned; drawing/pad verification pending; Function (none) -> 5 V / 0.5 A non-isolated DC/DC module; Height 17.5 -> 17.5 mm nominal; JLCPCB Status (none) -> No verified JLCPCB ID; source or consign; LCSC (none) -> UNVERIFIED; MPN (none) -> 173950575; Operating Temperature See datasheet -> -40 to +85 C (derated); Supplier Data Checked (none) -> UNDATED legacy record; Supplier Source (none) -> Legacy schematic record; exact supplier listing verificatio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; Temp Basis (none) -> Ambient with load derating; Temp Checked (none) -> 2026-10-03; Temp Max (degC) (none) -> 85; Temp Min (degC) (none) -> -40; Temp Source (none) -> https://www.we-online.com/components/products/datasheet/173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; Temp Status (none) -> Manufacturer rating recorded; system requirement pending
- PS2, PS6: Assembly (none) -> FIT; BOM Status (none) -> PART IDENTIFIED; sourcing/footprint review pending; Footprint Status (none) -> Assigned; drawing/pad verification pending; Function (none) -> Non-isolated 6.5 V SSI preregulator, 0.5 A; JLCPCB Status (none) -> No verified JLCPCB ID; source or consign; LCSC (none) -> UNVERIFIED; MANUFACTURER RECOM -> RECOM Power; MPN (none) -> R-78HB6.5-0.5; Operating Temperature (none) -> -40 to +85 C (derated); Supplier Data Checked (none) -> UNDATED legacy record; Supplier Source (none) -> Legacy schematic record; exact supplier listing verificatio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; Temp Basis (none) -> Ambient with load derating; Temp Checked (none) -> 2026-10-03; Temp Max (degC) (none) -> 85; Temp Min (degC) (none) -> -40; Temp Source (none) -> https://recom-power.com/pdf/Innoline/R-78HB-0.5.pdf; Temp Status (none) -> Manufacturer rating recorded; system requirement pending
- PS4: Assembly (none) -> FIT; BOM Review (none) -> 100 C endpoint requires load derating; verify stack load, s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; BOM Status (none) -> PART IDENTIFIED; sourcing/footprint review pending; Footprint Status (none) -> Assigned; drawing/pad verification pending; Function (none) -> REC10K-4805SAW_H2; JLCPCB Status (none) -> No verified JLCPCB ID; source or consign; LCSC (none) -> UNVERIFIED; MANUFACTURER Recom Power -> RECOM Power; MF Recom Power -> RECOM Power; MPN (none) -> REC10K-4805SAW/H2; Operating Temperature See datasheet -> -40 to +100 C (derated); Supplier Data Checked (none) -> UNDATED legacy record; Supplier Source (none) -> Legacy schematic record; exact supplier listing verificatio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; Temp Basis (none) -> Ambient with load derating; Temp Checked (none) -> 2026-10-03; Temp Max (degC) (none) -> 100; Temp Min (degC) (none) -> -40; Temp Source (none) -> https://recom-power.com/pdf/Econoline/REC10K-AW.pdf; Temp Status (none) -> Manufacturer rating recorded; system requirement pending
- PS5: Assembly (none) -> FIT; BOM Status (none) -> HOLD: 5 V supply architecture review; Footprint Status (none) -> Assigned; drawing/pad verification pending; Function (none) -> 5 V / 0.5 A non-isolated DC/DC module; Height 17.5 -> 17.5 mm nominal; JLCPCB Status (none) -> No verified JLCPCB ID; source or consign; LCSC (none) -> UNVERIFIED; MPN (none) -> 173950575; Operating Temperature See datasheet -> -40 to +85 C (derated); Supplier Data Checked (none) -> UNDATED legacy record; Supplier Source (none) -> Legacy schematic record; exact supplier listing verificatio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; Temp Basis (none) -> Ambient with load derating; Temp Checked (none) -> 2026-10-03; Temp Max (degC) (none) -> 85; Temp Min (degC) (none) -> -40; Temp Source (none) -> https://www.we-online.com/components/products/datasheet/173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; Temp Status (none) -> Manufacturer rating recorded; system requirement pending
- U14: Assembly (none) -> FIT; BOM Review (none) -> Keep current procurement field R05CTE05S-CT and schematic v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; BOM Status (none) -> REVIEW: -CT procurement suffix versus -R value; Footprint Status (none) -> Assigned; drawing/pad verification pending; Function (none) -> R05CTE05S-R; JLCPCB Status (none) -> Historical ID; recheck exact part and assembly availability; MPN (none) -> R05CTE05S-CT; Operating Temperature -40 to +125 C (derating applies) -> -40 to +125 C; Supplier Data Checked (none) -> UNDATED legacy record; Supplier Source (none) -> Legacy schematic record; exact supplier listing verificatio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; Temp Basis (none) -> Legacy rating; ambient/junction basis unverified; Temp Max (degC) (none) -> 125; Temp Min (degC) (none) -> -40; Temp Source (none) -> Legacy schematic field; primary-source verification pending; Temp Status (none) -> Inherited rating; system requirement pending
- U23, U25: Assembly (none) -> FIT; BOM Status (none) -> PART IDENTIFIED; sourcing/footprint review pending; Footprint Status (none) -> Assigned; drawing/pad verification pending; Function (none) -> TPS7A2450DBVR; JLCPCB Status (none) -> Historical ID; recheck exact part and assembly availability; MPN (none) -> TPS7A2450DBVR; Supplier Data Checked (none) -> UNDATED legacy record; Supplier Source (none) -> Legacy schematic record; exact supplier listing verificatio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; Temp Basis (none) -> Legacy rating; ambient/junction basis unverified; Temp Max (degC) (none) -> 125; Temp Min (degC) (none) -> -40; Temp Source (none) -> Legacy schematic field; primary-source verification pending; Temp Status (none) -> Inherited rating; system requirement pending
