File: LTC4364.kicad_sch (KiCad schematic)
At the start: 27 parts, among them Q14 IRFS4115TRLPBF, Q15 IRFS4115TRLPBF, Q16 SSM3K361R,LF, U4 LTC4364IS-2-PBF

Commit message: Redesign schematic for dual motor encoders
Other:
- note added: "Surge / ideal-diode controller"
Changed lines of the file:
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@@
 		(title "Elevation Control_Gigabit")
 		(date "2026-09-01")
-		(rev "Sep_2026_V1")
+		(rev "P3 REVIEW")
 		(company "Starspec")
 		(comment 4 "Mauro M. Coutinho")
@@
 		)
 	)
+	(text "Surge / ideal-diode controller"
+		(exclude_from_sim no)
+		(at 234.95 78.74 0)
+		(effects
+			(font
+				(size 1.27 1.27)
+			)
+		)
+	)
 	(text "Current sense resistor\n1%, 2512 package, 0.5 W or 1 W\nRoute SENSE/OUT as Kelvin traces to the resistor pads\n10 mOhms = 5A"
 		(exclude_from_sim no)
@@
 		(property "ALT_LCSC" "C6497281"
 			(at 204.47 189.23 0)
-			(effects (font (size 1.27 1.27)) (hide yes))
+			(effects
+				(font
+					(size 1.27 1.27)
+				)
+				(hide yes)
+			)
 		)
 		(property "ALT_MANUFACTURER_PART_NUMBER" "SSM3K361R,LXHF"
 			(at 204.47 189.23 0)
-			(effects (font (size 1.27 1.27)) (hide yes))
+			(effects
+				(font
+					(size 1.27 1.27)
+				)
+				(hide yes)
+			)
 		)
 		(pin "2"
@@
 		(property "ALT_LCSC" "C20564982"
 			(at 198.12 166.37 0)
-			(effects (font (size 1.27 1.27)) (hide yes))
+			(effects
+				(font
+					(size 1.27 1.27)
+				)
+				(hide yes)
+			)
 		)
 		(property "ALT_MANUFACTURER_PART_NUMBER" "MMSZ4699-HE3_A-08"
 			(at 198.12 166.37 0)
-			(effects (font (size 1.27 1.27)) (hide yes))
+			(effects
+				(font
+					(size 1.27 1.27)
+				)
+				(hide yes)
+			)
 		)
 		(property "Sim.Device" "D"

Commit message: Preserve P5 equal-size placement, controller stack and native BOM
Parts:
- C15: Assembly (none) -> FIT; BOM Status (none) -> PART IDENTIFIED; sourcing/footprint review pending; Footprint Status (none) -> Assigned; drawing/pad verification pending; Function (none) -> Unpolarized capacitor; JLCPCB Status (none) -> Historical ID; recheck exact part and assembly availability; MPN (none) -> CL21B103KCANNNC; Supplier Data Checked (none) -> UNDATED legacy record; Supplier Source (none) -> Legacy schematic record; exact supplier listing verificatio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; Temp Basis (none) -> Legacy rating; ambient/junction basis unverified; Temp Max (degC) (none) -> 125; Temp Min (degC) (none) -> -55; Temp Source (none) -> Legacy schematic field; primary-source verification pending; Temp Status (none) -> Inherited rating; system requirement pending
- C18: Assembly (none) -> FIT; BOM Status (none) -> PART IDENTIFIED; sourcing/footprint review pending; Footprint Status (none) -> Assigned; drawing/pad verification pending; Function (none) -> Unpolarized capacitor; JLCPCB Status (none) -> Historical ID; recheck exact part and assembly availability; MPN (none) -> CL21B104KCFNNNE; Supplier Data Checked (none) -> UNDATED legacy record; Supplier Source (none) -> Legacy schematic record; exact supplier listing verificatio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; Temp Basis (none) -> Legacy rating; ambient/junction basis unverified; Temp Max (degC) (none) -> 125; Temp Min (degC) (none) -> -55; Temp Source (none) -> Legacy schematic field; primary-source verification pending; Temp Status (none) -> Inherited rating; system requirement pending
- C19: Assembly (none) -> FIT; BOM Status (none) -> PART IDENTIFIED; sourcing/footprint review pending; Footprint Status (none) -> Assigned; drawing/pad verification pending; Function (none) -> Unpolarized capacitor; JLCPCB Status (none) -> Historical ID; recheck exact part and assembly availability; MPN (none) -> GCM31C5C1H104FA16L; Supplier Data Checked (none) -> UNDATED legacy record; Supplier Source (none) -> Legacy schematic record; exact supplier listing verificatio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; Temp Basis (none) -> Legacy rating; ambient/junction basis unverified; Temp Max (degC) (none) -> 125; Temp Min (degC) (none) -> -55; Temp Source (none) -> Legacy schematic field; primary-source verification pending; Temp Status (none) -> Inherited rating; system requirement pending
- C29, C30, C31, C32: Assembly (none) -> FIT; BOM Status (none) -> PART IDENTIFIED; sourcing/footprint review pending; Footprint Status (none) -> Assigned; drawing/pad verification pending; Function (none) -> Unpolarized capacitor; JLCPCB Status (none) -> Historical ID; recheck exact part and assembly availability; MPN (none) -> FS55X106K101EHG; Supplier Data Checked (none) -> UNDATED legacy record; Supplier Source (none) -> Legacy schematic record; exact supplier listing verificatio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; Temp Basis (none) -> Legacy rating; ambient/junction basis unverified; Temp Max (degC) (none) -> 125; Temp Min (degC) (none) -> -55; Temp Source (none) -> Legacy schematic field; primary-source verification pending; Temp Status (none) -> Inherited rating; system requirement pending
- D12: Assembly (none) -> FIT; BOM Status (none) -> REVIEW: temperature evidence; Footprint Status (none) -> Assigned; drawing/pad verification pending; Function (none) -> DIODE ZENER 68V 500MW SMA; JLCPCB Status (none) -> Historical ID; recheck exact part and assembly availability; MPN (none) -> CMZ5945B TR13 PBFREE; Operating Temperature See datasheet -> UNVERIFIED; Supplier Data Checked (none) -> UNDATED legacy record; Supplier Source (none) -> Legacy schematic record; exact supplier listing verificatio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; Temp Basis (none) -> Primary-source verification pending; Temp Max (degC) (none) -> UNVERIFIED; Temp Min (degC) (none) -> UNVERIFIED; Temp Status (none) -> UNVERIFIED
- D5: Assembly (none) -> FIT; BOM Review (none) -> Legacy datasheet is for Littelfuse but MPN/manufacturer spe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; BOM Status (none) -> REVIEW: legacy datasheet/manufacturer mismatch; Footprint Status (none) -> Assigned; drawing/pad verification pending; Function (none) -> 400W bidirectional Transient Voltage Suppressor, 70.0Vr, SM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; JLCPCB Status (none) -> Historical ID; recheck exact part and assembly availability; MPN (none) -> SMAJ70CA-TR; Supplier Data Checked (none) -> UNDATED legacy record; Supplier Source (none) -> Legacy schematic record; exact supplier listing verificatio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; Temp Basis (none) -> Legacy rating; ambient/junction basis unverified; Temp Max (degC) (none) -> 150; Temp Min (degC) (none) -> -55; Temp Source (none) -> Legacy schematic field; primary-source verification pending; Temp Status (none) -> Legacy rating unverified; exact manufacturer datasheet requ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
- D6: Assembly (none) -> FIT; BOM Status (none) -> REVIEW: temperature evidence; Footprint Status (none) -> Assigned; drawing/pad verification pending; Function (none) -> Zener Diode 12 V 500 mW ±5% Surface Mount SOD-123; JLCPCB Status (none) -> Historical ID; recheck exact part and assembly availability; MPN (none) -> BZT52C12; Operating Temperature See datasheet -> UNVERIFIED; Supplier Data Checked (none) -> UNDATED legacy record; Supplier Source (none) -> Legacy schematic record; exact supplier listing verificatio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; Temp Basis (none) -> Primary-source verification pending; Temp Max (degC) (none) -> UNVERIFIED; Temp Min (degC) (none) -> UNVERIFIED; Temp Status (none) -> UNVERIFIED
- D7: Assembly (none) -> FIT; BOM Review (none) -> Legacy datasheet points to ST ESDAL rather than selected on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; BOM Status (none) -> REVIEW: legacy datasheet/manufacturer mismatch; Footprint Status (none) -> Assigned; drawing/pad verification pending; Function (none) -> TVS Diode Array, 5.5V Standoff, 2 Channels, SOT23; JLCPCB Status (none) -> Historical ID; recheck exact part and assembly availability; MPN (none) -> MMBZ15VALT1G; Supplier Data Checked (none) -> UNDATED legacy record; Supplier Source (none) -> Legacy schematic record; exact supplier listing verificatio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; Temp Basis (none) -> Legacy rating; ambient/junction basis unverified; Temp Max (degC) (none) -> 150; Temp Min (degC) (none) -> -55; Temp Source (none) -> Legacy schematic field; primary-source verification pending; Temp Status (none) -> Legacy rating unverified; exact manufacturer datasheet requ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
- D9: Assembly (none) -> FIT; BOM Review (none) -> Legacy Vishay datasheet does not substantiate selected Semt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; BOM Status (none) -> REVIEW: legacy datasheet/manufacturer mismatch; Footprint Status (none) -> Assigned; drawing/pad verification pending; Function (none) -> 75V 0.15A Fast Switching Diode, SOD-123; JLCPCB Status (none) -> Historical ID; recheck exact part and assembly availability; MPN (none) -> 1N4148W; Operating Temperature See datasheet -> UNVERIFIED; Supplier Data Checked (none) -> UNDATED legacy record; Supplier Source (none) -> Legacy schematic record; exact supplier listing verificatio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; Temp Basis (none) -> Primary-source verification pending; Temp Max (degC) (none) -> UNVERIFIED; Temp Min (degC) (none) -> UNVERIFIED; Temp Status (none) -> Legacy rating unverified; exact manufacturer datasheet requ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
- Q14, Q15: Assembly (none) -> FIT; BOM Review (none) -> Absolute junction limits are not an ambient operating ratin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; BOM Status (none) -> PART IDENTIFIED; sourcing/footprint review pending; Footprint Status (none) -> Assigned; drawing/pad verification pending; Function (none) -> IRFS4115TRLPBF; JLCPCB Status (none) -> Historical ID; recheck exact part and assembly availability; MPN (none) -> IRFS4115TRLPBF; Operating Temperature See datasheet -> -55 to +175 C (Tj); Supplier Data Checked (none) -> UNDATED legacy record; Supplier Source (none) -> Legacy schematic record; exact supplier listing verificatio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; Temp Basis (none) -> Junction absolute limits; thermal/SOA design required; Temp Checked (none) -> 2026-10-03; Temp Max (degC) (none) -> 175; Temp Min (degC) (none) -> -55; Temp Source (none) -> https://www.infineon.com/assets/row/public/documents/24/49/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; Temp Status (none) -> Absolute junction limits only; ambient operating range unre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
- Q16: Assembly (none) -> FIT; BOM Status (none) -> REVIEW: temperature evidence; Footprint Status (none) -> Assigned; drawing/pad verification pending; Function (none) -> SSM3K361R,LF; JLCPCB Status (none) -> Historical ID; recheck exact part and assembly availability; MPN (none) -> SSM3K361R,LF; Operating Temperature See datasheet -> UNVERIFIED; Supplier Data Checked (none) -> UNDATED legacy record; Supplier Source (none) -> Legacy schematic record; exact supplier listing verificatio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; Temp Basis (none) -> Primary-source verification pending; Temp Max (degC) (none) -> UNVERIFIED; Temp Min (degC) (none) -> UNVERIFIED; Temp Status (none) -> UNVERIFIED
- R10: Assembly (none) -> FIT; BOM Status (none) -> PART IDENTIFIED; sourcing/footprint review pending; Footprint Status (none) -> Assigned; drawing/pad verification pending; Function (none) -> Resistor; JLCPCB Status (none) -> Historical ID; recheck exact part and assembly availability; MPN (none) -> RT0805BRD07205KL; Operating Temperature See datasheet -> -55 to +155 C; Power (none) -> 0.125 W at 70 C; Supplier Data Checked (none) -> UNDATED legacy record; Supplier Source (none) -> Legacy schematic record; exact supplier listing verificatio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; TCR (none) -> 25 ppm/C; Temp Basis (none) -> Operating; power derates above 70 C; Temp Checked (none) -> 2026-10-03; Temp Max (degC) (none) -> 155; Temp Min (degC) (none) -> -55; Temp Source (none) -> https://www.yageogroup.com/content/datasheet/asset/file/PYU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; Temp Status (none) -> Manufacturer rating recorded; system requirement pending; Tolerance (none) -> 0.1%
- R12: Assembly (none) -> FIT; BOM Status (none) -> PART IDENTIFIED; sourcing/footprint review pending; Footprint Status (none) -> Assigned; drawing/pad verification pending; Function (none) -> Resistor; JLCPCB Status (none) -> Historical ID; recheck exact part and assembly availability; MPN (none) -> RC0805FR-07100RL; Supplier Data Checked (none) -> UNDATED legacy record; Supplier Source (none) -> Legacy schematic record; exact supplier listing verificatio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; Temp Basis (none) -> Legacy rating; ambient/junction basis unverified; Temp Max (degC) (none) -> 155; Temp Min (degC) (none) -> -55; Temp Source (none) -> Legacy schematic field; primary-source verification pending; Temp Status (none) -> Inherited rating; system requirement pending
- R13: Assembly (none) -> FIT; BOM Status (none) -> PART IDENTIFIED; sourcing/footprint review pending; Footprint Status (none) -> Assigned; drawing/pad verification pending; Function (none) -> Resistor; JLCPCB Status (none) -> Historical ID; recheck exact part and assembly availability; MPN (none) -> RC0805FR-072K2L; Supplier Data Checked (none) -> UNDATED legacy record; Supplier Source (none) -> Legacy schematic record; exact supplier listing verificatio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; Temp Basis (none) -> Legacy rating; ambient/junction basis unverified; Temp Max (degC) (none) -> 155; Temp Min (degC) (none) -> -55; Temp Source (none) -> Legacy schematic field; primary-source verification pending; Temp Status (none) -> Inherited rating; system requirement pending
- R14: Assembly (none) -> FIT; BOM Status (none) -> PART IDENTIFIED; sourcing/footprint review pending; Footprint Status (none) -> Assigned; drawing/pad verification pending; Function (none) -> Resistor; JLCPCB Status (none) -> Historical ID; recheck exact part and assembly availability; MPN (none) -> RT0805BRD07523KL; Operating Temperature See datasheet -> -55 to +155 C; Power (none) -> 0.125 W at 70 C; Supplier Data Checked (none) -> UNDATED legacy record; Supplier Source (none) -> Legacy schematic record; exact supplier listing verificatio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; TCR (none) -> 25 ppm/C; Temp Basis (none) -> Operating; power derates above 70 C; Temp Checked (none) -> 2026-10-03; Temp Max (degC) (none) -> 155; Temp Min (degC) (none) -> -55; Temp Source (none) -> https://www.yageogroup.com/content/datasheet/asset/file/PYU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; Temp Status (none) -> Manufacturer rating recorded; system requirement pending; Tolerance (none) -> 0.1%
- R15: Assembly (none) -> FIT; BOM Status (none) -> PART IDENTIFIED; sourcing/footprint review pending; Footprint Status (none) -> Assigned; drawing/pad verification pending; Function (none) -> Resistor; JLCPCB Status (none) -> Historical ID; recheck exact part and assembly availability; MPN (none) -> RT0805BRD0727K4L; Operating Temperature See datasheet -> -55 to +155 C; Power (none) -> 0.125 W at 70 C; Supplier Data Checked (none) -> UNDATED legacy record; Supplier Source (none) -> Legacy schematic record; exact supplier listing verificatio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; TCR (none) -> 25 ppm/C; Temp Basis (none) -> Operating; power derates above 70 C; Temp Checked (none) -> 2026-10-03; Temp Max (degC) (none) -> 155; Temp Min (degC) (none) -> -55; Temp Source (none) -> https://www.yageogroup.com/content/datasheet/asset/file/PYU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; Temp Status (none) -> Manufacturer rating recorded; system requirement pending; Tolerance (none) -> 0.1%
- R16, R8: Assembly (none) -> FIT; BOM Status (none) -> PART IDENTIFIED; sourcing/footprint review pending; Footprint Status (none) -> Assigned; drawing/pad verification pending; Function (none) -> Resistor; JLCPCB Status (none) -> Historical ID; recheck exact part and assembly availability; MPN (none) -> RC0805FR-0710KL; Supplier Data Checked (none) -> UNDATED legacy record; Supplier Source (none) -> Legacy schematic record; exact supplier listing verificatio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; Temp Basis (none) -> Legacy rating; ambient/junction basis unverified; Temp Max (degC) (none) -> 155; Temp Min (degC) (none) -> -55; Temp Source (none) -> Legacy schematic field; primary-source verification pending; Temp Status (none) -> Inherited rating; system requirement pending
- R17: Assembly (none) -> FIT; BOM Status (none) -> REVIEW: temperature evidence; Footprint Status (none) -> Assigned; drawing/pad verification pending; Function (none) -> Resistor; JLCPCB Status (none) -> Historical ID; recheck exact part and assembly availability; MPN (none) -> PTFR0805Q4K02P9; Operating Temperature See datasheet -> UNVERIFIED; Supplier Data Checked (none) -> UNDATED legacy record; Supplier Source (none) -> Legacy schematic record; exact supplier listing verificatio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; Temp Basis (none) -> Primary-source verification pending; Temp Max (degC) (none) -> UNVERIFIED; Temp Min (degC) (none) -> UNVERIFIED; Temp Status (none) -> UNVERIFIED
- R6: Assembly (none) -> FIT; BOM Status (none) -> PART IDENTIFIED; sourcing/footprint review pending; Footprint Status (none) -> Assigned; drawing/pad verification pending; Function (none) -> Resistor; JLCPCB Status (none) -> Historical ID; recheck exact part and assembly availability; MPN (none) -> RC0805FR-0710RL; Supplier Data Checked (none) -> UNDATED legacy record; Supplier Source (none) -> Legacy schematic record; exact supplier listing verificatio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; Temp Basis (none) -> Legacy rating; ambient/junction basis unverified; Temp Max (degC) (none) -> 155; Temp Min (degC) (none) -> -55; Temp Source (none) -> Legacy schematic field; primary-source verification pending; Temp Status (none) -> Inherited rating; system requirement pending
- R63: Assembly (none) -> FIT; BOM Status (none) -> PART IDENTIFIED; sourcing/footprint review pending; Footprint Status (none) -> Assigned; drawing/pad verification pending; Function (none) -> Resistor; JLCPCB Status (none) -> Historical ID; recheck exact part and assembly availability; MPN (none) -> RC0805FR-07100KL; Supplier Data Checked (none) -> UNDATED legacy record; Supplier Source (none) -> Legacy schematic record; exact supplier listing verificatio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; Temp Basis (none) -> Legacy rating; ambient/junction basis unverified; Temp Max (degC) (none) -> 155; Temp Min (degC) (none) -> -55; Temp Source (none) -> Legacy schematic field; primary-source verification pending; Temp Status (none) -> Inherited rating; system requirement pending
- R7: Assembly (none) -> FIT; BOM Status (none) -> PART IDENTIFIED; sourcing/footprint review pending; Footprint Status (none) -> Assigned; drawing/pad verification pending; Function (none) -> Resistor; JLCPCB Status (none) -> Historical ID; recheck exact part and assembly availability; MPN (none) -> WSL2512R0100FEA18; Supplier Data Checked (none) -> UNDATED legacy record; Supplier Source (none) -> Legacy schematic record; exact supplier listing verificatio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; Temp Basis (none) -> Legacy rating; ambient/junction basis unverified; Temp Max (degC) (none) -> 170; Temp Min (degC) (none) -> -65; Temp Source (none) -> Legacy schematic field; primary-source verification pending; Temp Status (none) -> Inherited rating; system requirement pending
- U4: Assembly (none) -> FIT; BOM Status (none) -> PART IDENTIFIED; sourcing/footprint review pending; Footprint Status (none) -> Assigned; drawing/pad verification pending; Function (none) -> LTC4364IS-2-PBF; JLCPCB Status (none) -> Historical ID; recheck exact part and assembly availability; MPN (none) -> LTC4364IS-2#PBF; Supplier Data Checked (none) -> UNDATED legacy record; Supplier Source (none) -> Legacy schematic record; exact supplier listing verificatio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; Temp Basis (none) -> Legacy rating; ambient/junction basis unverified; Temp Max (degC) (none) -> 125; Temp Min (degC) (none) -> -40; Temp Source (none) -> Legacy schematic field; primary-source verification pending; Temp Status (none) -> Inherited rating; system requirement pending
