File: Pivot_Encoder_Port.kicad_sch (KiCad schematic)
At the start: 34 parts, among them J12 CHASSIS / SHIELD, J20 DE9 FEMALE, U100 AM26LV32EIDR, U101 ISO7760FDWR, U102 TPD2E2U06QDBZRQ1, U103 TPD2E2U06QDBZRQ1, U104 TPD2E2U06QDBZRQ1, U105 TLV75533PDBVR

Commit message: Preserve P5 equal-size placement, controller stack and native BOM
Parts:
- C110: Assembly (none) -> FIT; BOM Review (none) -> 1210, 10 uF nominal. Verify at least 3.3 uF effective at ma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; BOM Status (none) -> HOLD: DC-bias capacitance and converter arrangement; Dielectric (none) -> X7R; Footprint Status (none) -> Assigned; drawing/pad verification pending; Function (none) -> Encoder converter input capacitor; candidate pending DC-bia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; Height (none) -> 2.80 mm max; JLCPCB Status (none) -> No verified JLCPCB ID; source or consign; LCSC (none) -> UNVERIFIED; MPN (none) -> CGA6P1X7R2A106K250AC; Manufacturer (none) -> TDK; Operating Temperature (none) -> -55 to +125 C; Supplier Data Checked (none) -> UNDATED legacy record; Supplier Source (none) -> Legacy schematic record; exact supplier listing verificatio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; Temp Basis (none) -> Operating; Temp Checked (none) -> 2026-10-03; Temp Max (degC) (none) -> 125; Temp Min (degC) (none) -> -55; Temp Source (none) -> https://product.tdk.com/en/search/capacitor/ceramic/mlcc/in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; Temp Status (none) -> Manufacturer rating recorded; system requirement pending; Tolerance (none) -> 10%; Voltage (none) -> 100 V
- C111: Assembly (none) -> FIT; BOM Status (none) -> PART IDENTIFIED; sourcing/footprint review pending; Dielectric (none) -> X7R; Footprint Status (none) -> Assigned; drawing/pad verification pending; Function (none) -> Encoder 5 V output decoupling capacitor; Height (none) -> 1.40 mm max; JLCPCB Library (none) -> Extended; JLCPCB Status (none) -> Exact catalog match; stock not verified; LCSC (none) -> C95841; MPN (none) -> CL21B106KOQNNNE; Manufacturer (none) -> Samsung Electro-Mechanics; Operating Temperature (none) -> -55 to +125 C; Supplier Data Checked (none) -> 2026-10-03; Supplier Source (none) -> https://jlcpcb.com/partdetail/CL21B106KOQNNNE/C95841; Temp Basis (none) -> Operating; Temp Checked (none) -> 2026-10-03; Temp Max (degC) (none) -> 125; Temp Min (degC) (none) -> -55; Temp Source (none) -> https://product.samsungsem.com/mlcc/CL21B106KOQNNN.do; Temp Status (none) -> Manufacturer rating recorded; system requirement pending; Tolerance (none) -> 10%; Voltage (none) -> 16 V
- C112, C113, C114: Assembly (none) -> FIT; BOM Status (none) -> PART IDENTIFIED; sourcing/footprint review pending; Dielectric (none) -> X7R; DigiKey Part # (none) -> 445-14533-1-ND; DigiKey Status (none) -> VERIFIED; Footprint Status (none) -> Assigned; drawing/pad verification pending; Function (none) -> Unpolarized capacitor; JLCPCB Library (none) -> NOT_LISTED; JLCPCB Status (none) -> No verified JLCPCB ID; source or consign; JLCPCB Stock Snapshot (none) -> 0; LCSC (none) -> NOT_LISTED; MPN (none) -> C2012X7R1E105K085AB; Manufacturer (none) -> TDK; Operating Temperature (none) -> -55 to +125 C; Supplier Data Checked (none) -> 2026-09-18; Supplier Source (none) -> Legacy schematic record; exact supplier listing verificatio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; Temp Basis (none) -> Operating; Temp Max (degC) (none) -> 125; Temp Min (degC) (none) -> -55; Temp Source (none) -> https://product.tdk.com/en/search/capacitor/ceramic/mlcc/in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; Temp Status (none) -> Inherited rating; system requirement pending; Voltage (none) -> 25V
- C115, C116, C117: Assembly (none) -> FIT; BOM Status (none) -> PART IDENTIFIED; sourcing/footprint review pending; Footprint Status (none) -> Assigned; drawing/pad verification pending; Function (none) -> Unpolarized capacitor; JLCPCB Status (none) -> Historical ID; recheck exact part and assembly availability; LCSC (none) -> C28233; MPN (none) -> CL21B104KCFNNNE; Manufacturer (none) -> Samsung Electro-Mechanics; Operating Temperature (none) -> -55 to +125 C; Supplier Data Checked (none) -> UNDATED legacy record; Supplier Source (none) -> Legacy schematic record; exact supplier listing verificatio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; Temp Basis (none) -> Legacy rating; ambient/junction basis unverified; Temp Max (degC) (none) -> 125; Temp Min (degC) (none) -> -55; Temp Source (none) -> Legacy schematic field; primary-source verification pending; Temp Status (none) -> Inherited rating; system requirement pending
- C188: Assembly (none) -> FIT; BOM Status (none) -> PART IDENTIFIED; sourcing/footprint review pending; Dielectric (none) -> X7R; Footprint Status (none) -> Assigned; drawing/pad verification pending; Function (none) -> Field-to-chassis coupling capacitor, 1 nF; Height (none) -> 1.40 mm max; JLCPCB Library (none) -> UNVERIFIED; JLCPCB Status (none) -> LCSC exact match; JLC assembly availability unverified; LCSC (none) -> C2167549; MPN (none) -> C0805C102KDRACTU; Manufacturer (none) -> KEMET; Operating Temperature (none) -> -55 to +125 C; Supplier Data Checked (none) -> 2026-10-03; Supplier Source (none) -> https://www.lcsc.com/product-detail/C2167549.html; Temp Basis (none) -> Operating; Temp Checked (none) -> 2026-10-03; Temp Max (degC) (none) -> 125; Temp Min (degC) (none) -> -55; Temp Source (none) -> https://search.kemet.com/component-documentation/download/s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; Temp Status (none) -> Manufacturer rating recorded; system requirement pending; Tolerance (none) -> 10%; Voltage (none) -> 1000 V DC
- J12: Assembly (none) -> PCB feature - no purchased component; BOM Status (none) -> PCB FEATURE; Function (none) -> Wire solder pad; wire belongs to harness BOM; JLCPCB Status (none) -> N/A; LCSC (none) -> N/A; MPN (none) -> N/A; Manufacturer (none) -> N/A; Operating Temperature (none) -> N/A; Temp Basis (none) -> PCB feature; Temp Max (degC) (none) -> N/A; Temp Min (degC) (none) -> N/A; Temp Status (none) -> N/A; now left out of the parts list
- J20: Assembly (none) -> FIT; BOM Review (none) -> Same MPN as existing DE9 connectors. Verify exact pin grid,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; BOM Status (none) -> PART IDENTIFIED; sourcing/footprint review pending; Footprint Status (none) -> REVIEW: compare exact TE drawing to generic KiCad footprint; Function (none) -> DE9 female right-angle PCB connector; JLCPCB Library (none) -> UNVERIFIED; JLCPCB Status (none) -> LCSC exact match; JLC assembly availability unverified; LCSC (none) -> C305941; MPN (none) -> 5747844-4; Manufacturer (none) -> TE Connectivity; Operating Temperature (none) -> -55 to +105 C; Supplier Data Checked (none) -> 2026-10-03; Supplier Source (none) -> https://www.lcsc.com/de/product-detail/C305941.html; Temp Basis (none) -> Operating; Temp Checked (none) -> 2026-10-03; Temp Max (degC) (none) -> 105; Temp Min (degC) (none) -> -55; Temp Source (none) -> https://www.te.com/en/product-5747844-4.html; Temp Status (none) -> Manufacturer rating recorded; system requirement pending
- PS10: Assembly (none) -> FIT; BOM Review (none) -> Current schematic choice retained. No verified JLCPCB code.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; BOM Status (none) -> HOLD: 5 V supply architecture review; Footprint Status (none) -> Assigned; drawing/pad verification pending; Function (none) -> Non-isolated battery-to-5 V encoder converter, 0.5 A; Height (none) -> 17.5 mm nominal; JLCPCB Status (none) -> No verified JLCPCB ID; source or consign; LCSC (none) -> UNVERIFIED; MPN (none) -> R-78HB5.0-0.5; Manufacturer (none) -> RECOM Power; Operating Temperature (none) -> -40 to +85 C (derated); Supplier Data Checked (none) -> UNDATED legacy record; Supplier Source (none) -> Legacy schematic record; exact supplier listing verificatio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; Temp Basis (none) -> Ambient with load derating; Temp Checked (none) -> 2026-10-03; Temp Max (degC) (none) -> 85; Temp Min (degC) (none) -> -40; Temp Source (none) -> https://recom-power.com/pdf/Innoline/R-78HB-0.5.pdf; Temp Status (none) -> Manufacturer rating recorded; system requirement pending
- R100, R103, R106: Assembly (none) -> FIT; BOM Status (none) -> PART IDENTIFIED; sourcing/footprint review pending; Footprint Status (none) -> Assigned; drawing/pad verification pending; Function (none) -> Encoder differential-pair termination resistor; JLCPCB Library (none) -> UNVERIFIED; JLCPCB Status (none) -> LCSC exact match; JLC assembly availability unverified; LCSC (none) -> C4311641; MPN (none) -> ERJ-P08F1200V; Manufacturer (none) -> Panasonic; Operating Temperature (none) -> -55 to +155 C (derated); Power (none) -> 0.66 W nominal; temperature derating required; Supplier Data Checked (none) -> 2026-10-03; Supplier Source (none) -> https://www.lcsc.com/product-detail/chip-resistor-surface-m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; Temp Basis (none) -> Operating with power derating; Temp Checked (none) -> 2026-10-03; Temp Max (degC) (none) -> 155; Temp Min (degC) (none) -> -55; Temp Source (none) -> https://na.industrial.panasonic.com/products/resistors/smd-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; Temp Status (none) -> Manufacturer rating recorded; system requirement pending; Tolerance (none) -> 1%
- R101, R102, R104, R105, R107, R108: Assembly (none) -> FIT; BOM Status (none) -> PART IDENTIFIED; sourcing/footprint review pending; Footprint Status (none) -> Assigned; drawing/pad verification pending; Function (none) -> Resistor; JLCPCB Status (none) -> Historical ID; recheck exact part and assembly availability; LCSC (none) -> C114536; MPN (none) -> RC0805FR-07560RL; Manufacturer (none) -> Yageo; Operating Temperature (none) -> -55 to +155 C; Supplier Data Checked (none) -> UNDATED legacy record; Supplier Source (none) -> Legacy schematic record; exact supplier listing verificatio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; Temp Basis (none) -> Legacy rating; ambient/junction basis unverified; Temp Max (degC) (none) -> 155; Temp Min (degC) (none) -> -55; Temp Source (none) -> Legacy schematic field; primary-source verification pending; Temp Status (none) -> Inherited rating; system requirement pending
- R172: Assembly DNP -> DNP - not purchased; BOM Status (none) -> DNP; Footprint Status (none) -> Assigned; drawing/pad verification pending; Function (none) -> Resistor; JLCPCB Status (none) -> No verified JLCPCB ID; source or consign; LCSC (none) -> NOT SELECTED; MPN (none) -> NOT SELECTED - DNP; Manufacturer (none) -> NOT SELECTED; Operating Temperature (none) -> NOT SELECTED - DNP; Supplier Data Checked (none) -> UNDATED legacy record; Supplier Source (none) -> Legacy schematic record; exact supplier listing verificatio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; Temp Basis (none) -> Primary-source verification pending; Temp Max (degC) (none) -> N/A; Temp Min (degC) (none) -> N/A; Temp Status (none) -> NOT_EVALUATED_DNP
- TP20, TP21, TP22, TP23, TP24, TP25: Assembly (none) -> PCB feature - no purchased component; BOM Status (none) -> PCB FEATURE; Function (none) -> PCB test pad; JLCPCB Status (none) -> N/A; LCSC (none) -> N/A; MPN (none) -> N/A; Manufacturer (none) -> N/A; Operating Temperature (none) -> N/A; Temp Basis (none) -> PCB feature; Temp Max (degC) (none) -> N/A; Temp Min (degC) (none) -> N/A; Temp Status (none) -> N/A; now left out of the parts list
- U100: Assembly (none) -> FIT; BOM Status (none) -> PART IDENTIFIED; sourcing/footprint review pending; Footprint Status (none) -> Assigned; drawing/pad verification pending; Function (none) -> 3.3 V quad differential encoder receiver; JLCPCB Library (none) -> Extended; JLCPCB Status (none) -> Exact catalog match; stock not verified; LCSC (none) -> C527448; MPN (none) -> AM26LV32EIDR; Manufacturer (none) -> Texas Instruments; Operating Temperature (none) -> -40 to +85 C; Supplier Data Checked (none) -> 2026-10-03; Supplier Source (none) -> https://jlcpcb.com/partdetail/TexasInstruments-AM26LV32EIDR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; Temp Basis (none) -> Ambient; Temp Checked (none) -> 2026-10-03; Temp Max (degC) (none) -> 85; Temp Min (degC) (none) -> -40; Temp Source (none) -> https://www.ti.com/lit/ds/symlink/am26lv32e.pdf; Temp Status (none) -> Manufacturer rating recorded; system requirement pending
- U101: Assembly (none) -> FIT; BOM Status (none) -> PART IDENTIFIED; sourcing/footprint review pending; Footprint Status (none) -> Assigned; drawing/pad verification pending; Function (none) -> Six-channel encoder digital isolator, all channels toward M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; JLCPCB Library (none) -> UNVERIFIED; JLCPCB Status (none) -> LCSC exact match; JLC assembly availability unverified; LCSC (none) -> C2878538; MPN (none) -> ISO7760FDWR; Manufacturer (none) -> Texas Instruments; Operating Temperature (none) -> -55 to +125 C; Supplier Data Checked (none) -> 2026-10-03; Supplier Source (none) -> https://www.lcsc.com/product-detail/C2878538.html; Temp Basis (none) -> Ambient; Temp Checked (none) -> 2026-10-03; Temp Max (degC) (none) -> 125; Temp Min (degC) (none) -> -55; Temp Source (none) -> https://www.ti.com/lit/ds/symlink/iso7760.pdf; Temp Status (none) -> Manufacturer rating recorded; system requirement pending
- U102, U103, U104: Assembly (none) -> FIT; BOM Status (none) -> PART IDENTIFIED; sourcing/footprint review pending; Footprint Status (none) -> Assigned; drawing/pad verification pending; Function (none) -> Dual 5 V signal ESD protection; Height (none) -> 0.95; JLCPCB Status (none) -> Historical ID; recheck exact part and assembly availability; LCSC (none) -> C488151; MPN (none) -> TPD2E2U06QDBZRQ1; Manufacturer (none) -> Texas Instruments; Operating Temperature (none) -> -40 to +125 C; Supplier Data Checked (none) -> UNDATED legacy record; Supplier Source (none) -> Legacy schematic record; exact supplier listing verificatio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; Temp Basis (none) -> Legacy rating; ambient/junction basis unverified; Temp Max (degC) (none) -> 125; Temp Min (degC) (none) -> -40; Temp Source (none) -> Legacy schematic field; primary-source verification pending; Temp Status (none) -> Inherited rating; system requirement pending
- U105: Assembly (none) -> FIT; BOM Status (none) -> PART IDENTIFIED; sourcing/footprint review pending; Footprint Status (none) -> Assigned; drawing/pad verification pending; Function (none) -> 3.3 V LDO for both field-side encoder receivers; JLCPCB Library (none) -> Extended; JLCPCB Status (none) -> Exact catalog match; stock not verified; LCSC (none) -> C404027; MPN (none) -> TLV75533PDBVR; Manufacturer (none) -> Texas Instruments; Operating Temperature (none) -> -40 to +125 C (Tj); Supplier Data Checked (none) -> 2026-10-03; Supplier Source (none) -> https://jlcpcb.com/partdetail/TexasInstruments-TLV75533PDBV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; Temp Basis (none) -> Junction; ambient limit depends on dissipation; Temp Checked (none) -> 2026-10-03; Temp Max (degC) (none) -> 125; Temp Min (degC) (none) -> -40; Temp Source (none) -> https://www.ti.com/lit/ds/symlink/tlv755p.pdf; Temp Status (none) -> Manufacturer rating recorded; system requirement pending
