File: Pivot_Encoder_Star.kicad_sch (KiCad schematic)
At the start: 19 parts, among them J21 DE9 FEMALE, U110 AM26LV32EIDR, U112 TPD2E2U06QDBZRQ1, U113 TPD2E2U06QDBZRQ1, U114 TPD2E2U06QDBZRQ1

Commit message: Preserve P5 equal-size placement, controller stack and native BOM
Parts:
- C140: Assembly (none) -> FIT; BOM Review (none) -> 1210, 10 uF nominal. Verify at least 3.3 uF effective at ma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; BOM Status (none) -> HOLD: DC-bias capacitance and converter arrangement; Dielectric (none) -> X7R; Footprint Status (none) -> Assigned; drawing/pad verification pending; Function (none) -> Encoder converter input capacitor; candidate pending DC-bia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; Height (none) -> 2.80 mm max; JLCPCB Status (none) -> No verified JLCPCB ID; source or consign; LCSC (none) -> UNVERIFIED; MPN (none) -> CGA6P1X7R2A106K250AC; Manufacturer (none) -> TDK; Operating Temperature (none) -> -55 to +125 C; Supplier Data Checked (none) -> UNDATED legacy record; Supplier Source (none) -> Legacy schematic record; exact supplier listing verificatio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; Temp Basis (none) -> Operating; Temp Checked (none) -> 2026-10-03; Temp Max (degC) (none) -> 125; Temp Min (degC) (none) -> -55; Temp Source (none) -> https://product.tdk.com/en/search/capacitor/ceramic/mlcc/in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; Temp Status (none) -> Manufacturer rating recorded; system requirement pending; Tolerance (none) -> 10%; Voltage (none) -> 100 V
- C141: Assembly (none) -> FIT; BOM Status (none) -> PART IDENTIFIED; sourcing/footprint review pending; Dielectric (none) -> X7R; Footprint Status (none) -> Assigned; drawing/pad verification pending; Function (none) -> Encoder 5 V output decoupling capacitor; Height (none) -> 1.40 mm max; JLCPCB Library (none) -> Extended; JLCPCB Status (none) -> Exact catalog match; stock not verified; LCSC (none) -> C95841; MPN (none) -> CL21B106KOQNNNE; Manufacturer (none) -> Samsung Electro-Mechanics; Operating Temperature (none) -> -55 to +125 C; Supplier Data Checked (none) -> 2026-10-03; Supplier Source (none) -> https://jlcpcb.com/partdetail/CL21B106KOQNNNE/C95841; Temp Basis (none) -> Operating; Temp Checked (none) -> 2026-10-03; Temp Max (degC) (none) -> 125; Temp Min (degC) (none) -> -55; Temp Source (none) -> https://product.samsungsem.com/mlcc/CL21B106KOQNNN.do; Temp Status (none) -> Manufacturer rating recorded; system requirement pending; Tolerance (none) -> 10%; Voltage (none) -> 16 V
- C142: Assembly (none) -> FIT; BOM Status (none) -> PART IDENTIFIED; sourcing/footprint review pending; Dielectric (none) -> X7R; DigiKey Part # (none) -> 445-14533-1-ND; DigiKey Status (none) -> VERIFIED; Footprint Status (none) -> Assigned; drawing/pad verification pending; Function (none) -> Unpolarized capacitor; JLCPCB Library (none) -> NOT_LISTED; JLCPCB Status (none) -> No verified JLCPCB ID; source or consign; JLCPCB Stock Snapshot (none) -> 0; LCSC (none) -> NOT_LISTED; MPN (none) -> C2012X7R1E105K085AB; Manufacturer (none) -> TDK; Operating Temperature (none) -> -55 to +125 C; Supplier Data Checked (none) -> 2026-09-18; Supplier Source (none) -> Legacy schematic record; exact supplier listing verificatio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; Temp Basis (none) -> Operating; Temp Max (degC) (none) -> 125; Temp Min (degC) (none) -> -55; Temp Source (none) -> https://product.tdk.com/en/search/capacitor/ceramic/mlcc/in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; Temp Status (none) -> Inherited rating; system requirement pending; Voltage (none) -> 25V
- C145: Assembly (none) -> FIT; BOM Status (none) -> PART IDENTIFIED; sourcing/footprint review pending; Footprint Status (none) -> Assigned; drawing/pad verification pending; Function (none) -> Unpolarized capacitor; JLCPCB Status (none) -> Historical ID; recheck exact part and assembly availability; LCSC (none) -> C28233; MPN (none) -> CL21B104KCFNNNE; Manufacturer (none) -> Samsung Electro-Mechanics; Operating Temperature (none) -> -55 to +125 C; Supplier Data Checked (none) -> UNDATED legacy record; Supplier Source (none) -> Legacy schematic record; exact supplier listing verificatio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; Temp Basis (none) -> Legacy rating; ambient/junction basis unverified; Temp Max (degC) (none) -> 125; Temp Min (degC) (none) -> -55; Temp Source (none) -> Legacy schematic field; primary-source verification pending; Temp Status (none) -> Inherited rating; system requirement pending
- J21: Assembly (none) -> FIT; BOM Review (none) -> Same MPN as existing DE9 connectors. Verify exact pin grid,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; BOM Status (none) -> PART IDENTIFIED; sourcing/footprint review pending; Footprint Status (none) -> REVIEW: compare exact TE drawing to generic KiCad footprint; Function (none) -> DE9 female right-angle PCB connector; JLCPCB Library (none) -> UNVERIFIED; JLCPCB Status (none) -> LCSC exact match; JLC assembly availability unverified; LCSC (none) -> C305941; MPN (none) -> 5747844-4; Manufacturer (none) -> TE Connectivity; Operating Temperature (none) -> -55 to +105 C; Supplier Data Checked (none) -> 2026-10-03; Supplier Source (none) -> https://www.lcsc.com/de/product-detail/C305941.html; Temp Basis (none) -> Operating; Temp Checked (none) -> 2026-10-03; Temp Max (degC) (none) -> 105; Temp Min (degC) (none) -> -55; Temp Source (none) -> https://www.te.com/en/product-5747844-4.html; Temp Status (none) -> Manufacturer rating recorded; system requirement pending
- PS11: Assembly (none) -> FIT; BOM Review (none) -> Current schematic choice retained. No verified JLCPCB code.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; BOM Status (none) -> HOLD: 5 V supply architecture review; Footprint Status (none) -> Assigned; drawing/pad verification pending; Function (none) -> Non-isolated battery-to-5 V encoder converter, 0.5 A; Height (none) -> 17.5 mm nominal; JLCPCB Status (none) -> No verified JLCPCB ID; source or consign; LCSC (none) -> UNVERIFIED; MPN (none) -> R-78HB5.0-0.5; Manufacturer (none) -> RECOM Power; Operating Temperature (none) -> -40 to +85 C (derated); Supplier Data Checked (none) -> UNDATED legacy record; Supplier Source (none) -> Legacy schematic record; exact supplier listing verificatio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; Temp Basis (none) -> Ambient with load derating; Temp Checked (none) -> 2026-10-03; Temp Max (degC) (none) -> 85; Temp Min (degC) (none) -> -40; Temp Source (none) -> https://recom-power.com/pdf/Innoline/R-78HB-0.5.pdf; Temp Status (none) -> Manufacturer rating recorded; system requirement pending
- R130, R133, R136: Assembly (none) -> FIT; BOM Status (none) -> PART IDENTIFIED; sourcing/footprint review pending; Footprint Status (none) -> Assigned; drawing/pad verification pending; Function (none) -> Encoder differential-pair termination resistor; JLCPCB Library (none) -> UNVERIFIED; JLCPCB Status (none) -> LCSC exact match; JLC assembly availability unverified; LCSC (none) -> C4311641; MPN (none) -> ERJ-P08F1200V; Manufacturer (none) -> Panasonic; Operating Temperature (none) -> -55 to +155 C (derated); Power (none) -> 0.66 W nominal; temperature derating required; Supplier Data Checked (none) -> 2026-10-03; Supplier Source (none) -> https://www.lcsc.com/product-detail/chip-resistor-surface-m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; Temp Basis (none) -> Operating with power derating; Temp Checked (none) -> 2026-10-03; Temp Max (degC) (none) -> 155; Temp Min (degC) (none) -> -55; Temp Source (none) -> https://na.industrial.panasonic.com/products/resistors/smd-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; Temp Status (none) -> Manufacturer rating recorded; system requirement pending; Tolerance (none) -> 1%
- R131, R132, R134, R135, R137, R138: Assembly (none) -> FIT; BOM Status (none) -> PART IDENTIFIED; sourcing/footprint review pending; Footprint Status (none) -> Assigned; drawing/pad verification pending; Function (none) -> Resistor; JLCPCB Status (none) -> Historical ID; recheck exact part and assembly availability; LCSC (none) -> C114536; MPN (none) -> RC0805FR-07560RL; Manufacturer (none) -> Yageo; Operating Temperature (none) -> -55 to +155 C; Supplier Data Checked (none) -> UNDATED legacy record; Supplier Source (none) -> Legacy schematic record; exact supplier listing verificatio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; Temp Basis (none) -> Legacy rating; ambient/junction basis unverified; Temp Max (degC) (none) -> 155; Temp Min (degC) (none) -> -55; Temp Source (none) -> Legacy schematic field; primary-source verification pending; Temp Status (none) -> Inherited rating; system requirement pending
- U110: Assembly (none) -> FIT; BOM Status (none) -> PART IDENTIFIED; sourcing/footprint review pending; Footprint Status (none) -> Assigned; drawing/pad verification pending; Function (none) -> 3.3 V quad differential encoder receiver; JLCPCB Library (none) -> Extended; JLCPCB Status (none) -> Exact catalog match; stock not verified; LCSC (none) -> C527448; MPN (none) -> AM26LV32EIDR; Manufacturer (none) -> Texas Instruments; Operating Temperature (none) -> -40 to +85 C; Supplier Data Checked (none) -> 2026-10-03; Supplier Source (none) -> https://jlcpcb.com/partdetail/TexasInstruments-AM26LV32EIDR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; Temp Basis (none) -> Ambient; Temp Checked (none) -> 2026-10-03; Temp Max (degC) (none) -> 85; Temp Min (degC) (none) -> -40; Temp Source (none) -> https://www.ti.com/lit/ds/symlink/am26lv32e.pdf; Temp Status (none) -> Manufacturer rating recorded; system requirement pending
- U112, U113, U114: Assembly (none) -> FIT; BOM Status (none) -> PART IDENTIFIED; sourcing/footprint review pending; Footprint Status (none) -> Assigned; drawing/pad verification pending; Function (none) -> Dual 5 V signal ESD protection; Height (none) -> 0.95; JLCPCB Status (none) -> Historical ID; recheck exact part and assembly availability; LCSC (none) -> C488151; MPN (none) -> TPD2E2U06QDBZRQ1; Manufacturer (none) -> Texas Instruments; Operating Temperature (none) -> -40 to +125 C; Supplier Data Checked (none) -> UNDATED legacy record; Supplier Source (none) -> Legacy schematic record; exact supplier listing verificatio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; Temp Basis (none) -> Legacy rating; ambient/junction basis unverified; Temp Max (degC) (none) -> 125; Temp Min (degC) (none) -> -40; Temp Source (none) -> Legacy schematic field; primary-source verification pending; Temp Status (none) -> Inherited rating; system requirement pending
