File: STM32.kicad_sch (KiCad schematic)
At the start: 14 parts, among them CN10 ESW-117-44-L-D, CN11 ESW-108-X-X-D, CN7 ESW-110-44-L-D, CN8 ESW-108-X-X-D, CN9 ESW-115-44-L-D, U1 NUCLEOH723ZG

Commit message: Redesign schematic for dual motor encoders
Connections:
- net STAR_ENC_A: now reaches CN7.01
- net STAR_ENC_A: now also U1.CN7_1 (D16/I2S_A_MCK)
- net PORT_ENC_A: now reaches CN7.10
- net PORT_ENC_A: now also U1.CN7_10 (D13/SPI_A_SCK)
- net STAR_ENC_B: now reaches CN7.11
- net STAR_ENC_B: now also U1.CN7_11 (D21/I2S_B_MCK)
- net PORT_ENC_B: now reaches CN7.15
- net PORT_ENC_B: now also U1.CN7_15 (D23/I2S_B_CK/SPI_B_SCK)
- net PORT_ENC_Z: now reaches U1.CN9_16 (D57/SAI_A_FS)
- net PORT_ENC_Z: now also CN9.16
- net STAR_ENC_Z: now reaches U1.CN9_22 (D60/SAI_B_SD)
- net STAR_ENC_Z: now also CN9.22
- net LH_BRAKE_RELEASE_CMD renamed PORT_BRAKE_RELEASE_CMD
- net LH_ENC_PRESET_N renamed PORT_ENC_PRESET_N
- net LH_SSI_CLK renamed PORT_SSI_CLK
- net LH_SSI_DATA renamed PORT_SSI_DATA
- net LH_STR8_DIR_CMD renamed PORT_STR8_DIR_CMD
- net LH_STR8_DISABLE renamed PORT_STR8_DISABLE
- net LH_STR8_FAULT renamed PORT_STR8_FAULT
- net LH_STR8_STEP_CMD renamed PORT_STR8_STEP_CMD
- net RH_BRAKE_RELEASE_CMD renamed STAR_BRAKE_RELEASE_CMD
- net RH_ENC_PRESET_N renamed STAR_ENC_PRESET_N
- net RH_SSI_CLK renamed STAR_SSI_CLK
- net RH_SSI_DATA renamed STAR_SSI_DATA
- net RH_STR8_DIR_CMD renamed STAR_STR8_DIR_CMD
- net RH_STR8_DISABLE renamed STAR_STR8_DISABLE
- net RH_STR8_FAULT renamed STAR_STR8_FAULT
- net RH_STR8_STEP_CMD renamed STAR_STR8_STEP_CMD
- no-connect marks 159 -> 147
Other:
- note added: "PIVOT ENCODERS: Port TIM2 PA5/PB3 (AF1); Star TIM3 PC6/PC7 (AF2). Index: PE4 / PE3 on EXTI4 / EXTI3. Retain all existing SSI and drive signals. Use SWD only; disable SWO trace on PB3. PA5 also drives the high-impedance D13 LED input."
- note added: "STM32H723 controller"
- moved on the sheet: CN7, U1A, U1B, U1C

Commit message: Preserve P5 equal-size placement, controller stack and native BOM
Parts:
- removed CN10: ESW-117-44-L-D, ESW-117-44-L-D:ESW-117-44-L-D, symbol ESW-117-44-L-D:ESW-117-44-L-D
- removed CN11, CN8: ESW-108-X-X-D, ESW-108-44-L-D:ESW-108-44-L-D, symbol ESW-108-44-L-D:ESW-108-X-X-D
- removed CN7: ESW-110-44-L-D, ESW-110-44-L-D:ESW-110-44-L-D, symbol ESW-110-44-L-D:ESW-110-44-L-D
- removed CN9: ESW-115-44-L-D, ESW-115-44-L-D:ESW-115-44-L-D, symbol ESW-115-44-L-D:ESW-115-44-L-D
- removed H1, H2, H3, H4: MountingHole, MountingHole:MountingHole_3.5mm, symbol Mechanical:MountingHole
- removed U1: NUCLEOH723ZG, NUCLEO-H723ZG:MODULE_NUCLEOH723ZG, symbol NUCLEOH723ZG:NUCLEOH723ZG_Daughterboard_Interface
- added H30, H31, H32, H33: M3 STACK SUPPORT, MountingHole:MountingHole_3.2mm_M3, symbol Mechanical:MountingHole
- added J30: SSW-115-01-S-D, Stack:Samtec_SSW-115-01-S-D, symbol Stack:Stack_2x15
- added J31: SSW-110-01-S-D, Stack:Samtec_SSW-110-01-S-D, symbol Stack:Stack_2x10
- added TP30: CTRL_NRST, TestPoint:TestPoint_Pad_D1.5mm, symbol Connector:TestPoint
- H5, H6, H7, H8: Assembly (none) -> PCB feature - no purchased component; BOM Status (none) -> PCB FEATURE; Function (none) -> PCB mounting hole; JLCPCB Status (none) -> N/A; LCSC (none) -> N/A; MPN (none) -> N/A; Manufacturer Mechanical -> N/A; Temp Basis (none) -> PCB feature; Temp Max (degC) (none) -> N/A; Temp Min (degC) (none) -> N/A; Temp Status (none) -> N/A
Connections:
- net +3V3_STM32: now also J30.29, J30.30
- net +5V_STM32: now also J30.25, J30.26
- net E_STOP_OK: now also J30.24
- net GND_STM32: now also J30.1, J30.11, J30.12, J30.2, J30.21, J30.22, J30.27, J30.28, J31.10, J31.20, J31.3, J31.4, J31.9
- net HOME_POS: now also J30.23
- net PORT_BRAKE_RELEASE_CMD: now also J30.19
- net PORT_ENC_A: now also J31.1
- net PORT_ENC_B: now also J31.2
- net PORT_ENC_PRESET_N: now also J30.17
- net PORT_ENC_Z: now also J31.7
- net PORT_SSI_CLK: now also J30.13
- net PORT_SSI_DATA: now also J30.15
- net PORT_STR8_DIR_CMD: now also J30.5
- net PORT_STR8_DISABLE: now also J30.7
- net PORT_STR8_FAULT: now also J30.9
- net PORT_STR8_STEP_CMD: now also J30.3
- net RX_CAN: now also J31.16
- net STAR_BRAKE_RELEASE_CMD: now also J30.20
- net STAR_ENC_A: now also J31.5
- net STAR_ENC_B: now also J31.6
- net STAR_ENC_PRESET_N: now also J30.18
- net STAR_ENC_Z: now also J31.8
- net STAR_SSI_CLK: now also J30.14
- net STAR_SSI_DATA: now also J30.16
- net STAR_STR8_DIR_CMD: now also J30.6
- net STAR_STR8_DISABLE: now also J30.8
- net STAR_STR8_FAULT: now also J30.10
- net STAR_STR8_STEP_CMD: now also J30.4
- net STM32_SCL: now also J31.11
- net STM32_SDA: now also J31.12
- net Silent_Mode: now also J31.17
- net TX_CAN: now also J31.15
- new net CTRL_NRST: J31.19, TP30.1
- new net PIVOT_MODBUS_DE: J31.18
- new net PIVOT_MODBUS_RX: J31.14
- new net PIVOT_MODBUS_TX: J31.13
- no-connect marks 147 -> 0
Other:
- note added: "Elevation top-side socket | 20 contacts"
- note added: "Elevation top-side socket | 30 contacts"
- note added: "J30 mates to J30; J31 mates to J31, same pin number to same pin number. 5 V: elevation PS4 -> controller. 3.3 V: controller buck -> elevation MCU-side logic. All signal returns use GND_STM32 / controller GND. No field return crosses these connectors. Mechanical definition: assembly/stack_interface.json. Nominal facing-board gap: 12 mm."
- note added: "MATCHED TWO-BOARD INTERFACE | J30 30 CONTACTS + J31 20 CONTACTS"
- note added: "P4.1: J31-13 TX, J31-14 RX, J31-18 DE -> isolated pivot Modbus RTU. These replace three P4 ground contacts. Mate only matching P4.1 boards. USART2: PD5 TX, PD6 RX, PD4 hardware DE, AF7. DE defaults low on carrier."
- note removed: "Nucleo power jumper: USB supply for USB-powered operation; E5V for daughterboard +5V_STM32. Select the matching jumper position on the Nucleo (user-confirmed arrangement)."
- note removed: "Nucleo-to-socket interface links"
- note removed: "PIVOT ENCODERS: Port TIM2 PA5/PB3 (AF1); Star TIM3 PC6/PC7 (AF2). Index: PE4 / PE3 on EXTI4 / EXTI3. Retain all existing SSI and drive signals. Use SWD only; disable SWO trace on PB3. PA5 also drives the high-impedance D13 LED input."
- note removed: "STM32H723 controller"
- note removed: "U1 models the daughterboard interface only: CN7-CN11. CN12, CN3, CN4, CN15 and CN16 are external Nucleo connectors, not daughterboard mating connections. U1 is excluded from PCB/BOM."
- title: Elevation Control_Gigabit -> Elevation to custom STM32 controller
- moved on the sheet: H5, H6, H7, H8

Commit message: Build P6 80x130 stack with redistributed SSI and stepper interfaces
Connections:
- net PORT_ENC_PRESET_N is gone; now on net TX_CAN: J30.17
- net PORT_SSI_CLK is gone; now on net GND_STM32: J30.13
- net PORT_SSI_DATA is gone; now on net STM32_SCL: J30.15
- net PORT_STR8_DIR_CMD is gone; now on net HOME_POS: J30.5
- net PORT_STR8_DISABLE is gone; now on net PORT_ENC_A: J30.7
- net PORT_STR8_FAULT is gone; now on net PORT_ENC_Z: J30.9
- net PORT_STR8_STEP_CMD is gone; now on net PORT_BRAKE_RELEASE_CMD: J30.3
- net STAR_ENC_PRESET_N is gone; now on net RX_CAN: J30.18
- net STAR_SSI_CLK is gone; now on net GND_STM32: J30.14
- net STAR_SSI_DATA is gone; now on net STM32_SDA: J30.16
- net STAR_STR8_DIR_CMD is gone; now on net E_STOP_OK: J30.6
- net STAR_STR8_DISABLE is gone; now on net PORT_ENC_B: J30.8
- net STAR_STR8_FAULT is gone; now on net STAR_ENC_A: J30.10
- net STAR_STR8_STEP_CMD is gone; now on net STAR_BRAKE_RELEASE_CMD: J30.4
- net +3V3_STM32: now also J30.27, J30.28; no longer J30.29, J30.30
- net CTRL_NRST: now also J30.23; no longer J31.19
- net E_STOP_OK: no longer J30.24
- net GND_STM32: now also J30.24, J30.29, J30.30; no longer J30.11, J30.12, J30.21, J30.22, J30.27, J30.28, J31.10, J31.20, J31.3, J31.4, J31.9
- net HOME_POS: no longer J30.23
- net PIVOT_MODBUS_DE: now also J30.22; no longer J31.18
- net PIVOT_MODBUS_RX: now also J30.21; no longer J31.14
- net PIVOT_MODBUS_TX: now also J30.20; no longer J31.13
- net PORT_BRAKE_RELEASE_CMD: no longer J30.19
- net PORT_ENC_A: no longer J31.1
- net PORT_ENC_B: no longer J31.2
- net PORT_ENC_Z: no longer J31.7
- net RX_CAN: no longer J31.16
- net STAR_BRAKE_RELEASE_CMD: no longer J30.20
- net STAR_ENC_A: no longer J31.5
- net STAR_ENC_B: now also J30.11; no longer J31.6
- net STAR_ENC_Z: now also J30.12; no longer J31.8
- net STM32_SCL: no longer J31.11
- net STM32_SDA: no longer J31.12
- net Silent_Mode: now also J30.19; no longer J31.17
- net TX_CAN: no longer J31.15
- new net +5V_ENC_PORT: J31.11, J31.12
- new net +5V_ENC_STAR: J31.17, J31.18
- new net +5V_FIELD: J31.5, J31.6
- new net +6.5V_ENC_PORT: J31.10, J31.9
- new net +6.5V_ENC_STAR: J31.15, J31.16
- new net -BATT: J31.1, J31.13, J31.14, J31.19, J31.2, J31.20, J31.3, J31.4, J31.7, J31.8
Other:
- note added: "J30 CLEAN LOGIC / STM32 GROUND"
- note added: "J31 FIELD SUPPLIES / -BATT RETURN SSI local 5 V and preregulator connections retained"
- note added: "Keep J30 clean copper separate from J31 field copper. No field current on STM32 grounds. Parallel supply contacts retained; confirm actual loads and derating before release."
- note added: "P6 STACK INTERFACE - incompatible with P4/P5 pinout"
- note removed: "Elevation top-side socket | 20 contacts"
- note removed: "Elevation top-side socket | 30 contacts"
- note removed: "J30 mates to J30; J31 mates to J31, same pin number to same pin number. 5 V: elevation PS4 -> controller. 3.3 V: controller buck -> elevation MCU-side logic. All signal returns use GND_STM32 / controller GND. No field return crosses these connectors. Mechanical definition: assembly/stack_interface.json. Nominal facing-board gap: 12 mm."
- note removed: "MATCHED TWO-BOARD INTERFACE | J30 30 CONTACTS + J31 20 CONTACTS"
- note removed: "P4.1: J31-13 TX, J31-14 RX, J31-18 DE -> isolated pivot Modbus RTU. These replace three P4 ground contacts. Mate only matching P4.1 boards. USART2: PD5 TX, PD6 RX, PD4 hardware DE, AF7. DE defaults low on carrier."
- moved on the sheet: H30, H31, H32, H33, H5, H6, H7, H8, J30, J31, TP30
